File: evse.kicad_pcb (KiCad board)
At the start: 2 copper layers, 100 x 100 mm, 27 parts, among them J2 KF128-2.54-4P, J3 KF128-2.54-2P, J4 T44009, J5 T44009, J6 T44009, J7 T44009, J8 T44009, J9 T44009, K1 HF186F/12-HCTF, K2 HF186F/12-HCTF, M1 MOV, M2 MOV, M3 MOV

Commit message: parts added
Parts:
- added C1: 12pF, Capacitor_SMD:C_0805_2012Metric, F.Cu at (84.1, 39.9)
- added C10: 10uF, Capacitor_SMD:C_0805_2012Metric, F.Cu at (-77.2, -52.0)
- added C11: 0.1uF, Capacitor_SMD:C_0805_2012Metric, F.Cu at (31.5, 58.7)
- added C12: 0.1uF, PCM_SparkFun-Capacitor:C_0805_2012Metric, F.Cu at (-77.2, -49.0)
- added C13: 10uF, Capacitor_SMD:C_0805_2012Metric, F.Cu at (-77.2, -46.0)
- added C15: 1.0uF, PCM_SparkFun-Capacitor:C_0805_2012Metric, F.Cu at (-77.2, -43.0)
- added C17: 10uF, PCM_SparkFun-Capacitor:C_0603_1608Metric_Polar, F.Cu at (-50.8, -46.4)
- added C18: 1.0uF, PCM_SparkFun-Capacitor:C_0805_2012Metric, F.Cu at (-85.2, -32.9)
- added C19: 0.1uF, PCM_SparkFun-Capacitor:C_0805_2012Metric, F.Cu at (-72.8, -55.1)
- added C2: 12pF, Capacitor_SMD:C_0805_2012Metric, F.Cu at (84.1, 46.9)
- added C20: 1.0uF, PCM_SparkFun-Capacitor:C_0805_2012Metric, F.Cu at (-72.8, -52.0)
- added C21: 0.1uF, PCM_SparkFun-Capacitor:C_0805_2012Metric, F.Cu at (-72.8, -49.0)
- added C22: 10uF, Capacitor_SMD:C_1206_3216Metric, F.Cu at (55.7, 54.7)
- added C23: 1.0uF, PCM_SparkFun-Capacitor:C_0805_2012Metric, F.Cu at (59.6, 51.5)
- added C24: 1.0uF, PCM_SparkFun-Capacitor:C_0805_2012Metric, F.Cu at (55.2, 51.4)
- added C26: 10uF, Capacitor_SMD:C_0805_2012Metric, F.Cu at (-72.8, -40.0)
- added C27: 0.1uF, PCM_SparkFun-Capacitor:C_0805_2012Metric, F.Cu at (-68.3, -55.1)
- added C28: 10uF, PCM_SparkFun-Capacitor:C_0805_2012Metric, F.Cu at (73.5, 61.9)
- added C29: 22uF, PCM_SparkFun-Capacitor:C_0805_2012Metric, F.Cu at (73.5, 57.7)
- added C3: 1.0uF, PCM_SparkFun-Capacitor:C_0805_2012Metric, F.Cu at (-81.7, -49.0)
- added C32: 0.1uF, Capacitor_SMD:C_0805_2012Metric, F.Cu at (83.2, 60.9)
- added C33: 22uF, PCM_SparkFun-Capacitor:C_0805_2012Metric, F.Cu at (73.5, 54.6)
- added C34: 100nF, Capacitor_SMD:C_0805_2012Metric, F.Cu at (111.1, 28.5)
- added C35: 0.1uF, Capacitor_SMD:C_0402_1005Metric, F.Cu at (-50.5, -43.8)
- added C4: 1.0uF, PCM_SparkFun-Capacitor:C_0805_2012Metric, F.Cu at (-81.7, -46.0)
- added C5: 10uF, Capacitor_SMD:C_0805_2012Metric, F.Cu at (-81.7, -43.0)
- added C6: 10uF, Capacitor_SMD:C_0805_2012Metric, F.Cu at (-81.7, -40.0)
- added C9: 1.0uF, PCM_SparkFun-Capacitor:C_0805_2012Metric, F.Cu at (-77.2, -55.1)
- added D11: AZ23C2V7, PCM_SparkFun-Semiconductor-Standard:SOT23-3, F.Cu at (31.5, 64.7)
- added D2: SS14, Diode_SMD:D_SOD-123, F.Cu at (104.9, 73.0)
- added D5: SS14, Diode_SMD:D_SOD-123, F.Cu at (83.8, 73.0)
- added FTDI1: Conn_01x06_Pin, OpenEVSE:FTDI_JST_PH_1x06_P2.00mm, B.Cu at (68.7, 24.2)
- added IC1: LF353, Package_SO:SOIC-8_3.9x4.9mm_P1.27mm, F.Cu at (-68.1, -35.1)
- added IC2: ATmega328P, PCM_SparkFun-Semiconductor-Standard:TQFP-32_7x7mm_P0.8mm, F.Cu at (92.0, 40.5)
- added J1: ISP, OpenEVSE:AVR_ISP_2x03_P2.54mm, B.Cu at (83.5, 26.0)
- added L1: BLM21PG331SN1D, PCM_SparkFun-Coil:0805, F.Cu at (-59.0, -40.1)
- added L2: 4.7uH, OpenEVSE:NR5040, F.Cu at (78.3, 56.5)
- added Q2: MMBT2222A, Package_TO_SOT_SMD:SOT-23, F.Cu at (88.0, 66.0)
- added Q3: MMBT2222A, Package_TO_SOT_SMD:SOT-23, F.Cu at (110.1, 66.0)
- added R1: 620, Resistor_SMD:R_0805_2012Metric, F.Cu at (-63.9, -55.1)
- added R10: 10k, Resistor_SMD:R_0805_2012Metric, F.Cu at (-59.5, -49.2)
- added R11: 220, Resistor_SMD:R_0805_2012Metric, F.Cu at (111.0, 61.0)
- added R21: 100k, Resistor_SMD:R_0805_2012Metric, F.Cu at (31.6, 61.5)
- added R22: 10k, Resistor_SMD:R_0805_2012Metric, F.Cu at (-55.1, -55.1)
- added R24: 220, Resistor_SMD:R_0805_2012Metric, F.Cu at (88.8, 61.0)
- added R25: 100k, Resistor_SMD:R_0805_2012Metric, F.Cu at (34.9, 60.6)
- added R26: 20R 1% 0.25W, Resistor_SMD:R_0805_2012Metric, F.Cu at (34.9, 64.7)
- added R27: 2, Resistor_SMD:R_0805_2012Metric, F.Cu at (-55.1, -49.2)
- added R31: 10k, Resistor_SMD:R_0805_2012Metric, F.Cu at (-55.1, -46.2)
- added R40: 4.7k, Resistor_SMD:R_0805_2012Metric, F.Cu at (106.3, 28.5)
- added R41: 4.7k, Resistor_SMD:R_0805_2012Metric, F.Cu at (108.7, 28.5)
- added R5: 56k, Resistor_SMD:R_0805_2012Metric, F.Cu at (-63.9, -52.1)
- added R6: 100k, Resistor_SMD:R_0805_2012Metric, F.Cu at (-63.9, -49.2)
- added R7: 200k, Resistor_SMD:R_0805_2012Metric, F.Cu at (-63.9, -46.2)
- added R8: 100k, Resistor_SMD:R_0805_2012Metric, F.Cu at (-59.5, -55.1)
- added R9: 100k, Resistor_SMD:R_0805_2012Metric, F.Cu at (-59.5, -52.1)
- added SH1: NetTie_2, OpenEVSE:SHORT_TOP-50, F.Cu at (-53.8, -43.5)
- added SH2: NetTie_2, OpenEVSE:SHORT_TOP-50, F.Cu at (-53.8, -41.1)
- added TVS1: P6SMB16CA, OpenEVSE:SMB, F.Cu at (-53.5, -30.1)
- added U1: AP63205WU, Package_TO_SOT_SMD:TSOT-23-6, F.Cu at (78.3, 61.9)
- added U2: TC1044S, Package_SO:SOIC-8_3.9x4.9mm_P1.27mm, F.Cu at (-97.3, -31.4)
- added U3: MCP9808, Package_SO:MSOP-8_3x3mm_P0.65mm, F.Cu at (108.7, 24.0)
- added Y1: 16MHz, PCM_SparkFun-Clock:Crystal_SMD_3.2x2.5mm, F.Cu at (84.8, 43.4)
- PS1: footprint Converter_ACDC:Converter_ACDC_MeanWell_IRM-10-xx_THT -> OpenEVSE:Converter_ACDC_MeanWell_IRM-10-12_THT
- moved ? 48.0 mm to (117.0, 23.0)
- moved G2 13.2 mm to (23.0, 23.0)
Routing:
- net +5V: track 0.00 -> 160.1 mm, vias 0 -> 3
- net MOSI: track 0.00 -> 64.8 mm
- net MISO: track 0.00 -> 45.7 mm
- net SCL: track 0.00 -> 39.4 mm, vias 0 -> 2
- net DC_RELAY_2: track 0.00 -> 35.2 mm
- net +12V: track 80.7 -> 114.4 mm
- net SDA: track 0.00 -> 32.3 mm, vias 0 -> 2
- net AMP_CT_SENSE: track 0.00 -> 19.0 mm
- net DC_RELAY_1: track 0.00 -> 15.4 mm
- net Net-(U1-SW): track 0.00 -> 14.7 mm
- net AMP_READ: track 0.00 -> 11.5 mm
- net DC_RELAY_C2: track 0.00 -> 10.0 mm
- net DC_RELAY_C1: track 0.00 -> 9.19 mm
- net Net-(C1-Pad1): track 0.00 -> 7.46 mm
- net Net-(IC2-XTAL2/PB7): track 0.00 -> 5.18 mm
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- added copper zone on F.Cu, net GND
- added copper zone on B.Cu, net UGND
- added copper zone on F.Cu, net UGND
Other:
- outline, holes or cut-outs redrawn
