File: evse.kicad_pcb (KiCad board)
At the start: 2 copper layers, 100 x 100 mm, 117 parts, among them IC1 LF353, IC2 ATmega328P, IC3 LM358, IC8 HCPL-2731S, J1 ISP, J4 T44009, J5 T44009, J6 T44009, J7 T44009, J8 T44009, J9 T44009, K1 HF186F/12-HCTF, K2 HF186F/12-HCTF, M1 MOV-20D431K, M2 MOV-20D431K, M3 MOV-20D431K, Q2 MMBT2222A, Q3 MMBT2222A, U1 AP63205WU, U2 TC1044S, U3 MCP9808, Y1 16MHz

Commit message: fix
Parts:
- removed the ? at (117.0, 23.0)
- removed the FID4 at (115.0, 26.0)
- removed the FID4 at (26.0, 26.0)
- removed G2: M01PTH, 1X01
- removed IC2: ATmega328P, PCM_SparkFun-Semiconductor-Standard:TQFP-32_7x7mm_P0.8mm
- added FID1: FIDUCIAL1X2, Fiducial:Fiducial_1mm_Mask2mm, F.Cu at (27.3, 26.5)
- added FID2: FIDUCIAL1X2, Fiducial:Fiducial_1mm_Mask2mm, F.Cu at (53.3, -15.3)
- added FID3: FIDUCIAL1X2, Fiducial:Fiducial_1mm_Mask2mm, F.Cu at (66.2, -14.8)
- added FID4: FIDUCIAL1X2, Fiducial:Fiducial_1mm_Mask2mm, F.Cu at (79.2, -14.3)
- added U$3: HOLE, coreEVSE:HOLE, F.Cu at (23.5, 23.6)
- added U$9: HOLE, coreEVSE:HOLE, F.Cu at (116.5, 23.6)
- added U4: ATmega328P-AU, PCM_JLCPCB:TQFP-32_7x7mm_P0.8mm, F.Cu at (72.7, 39.6)
- C1, C2: value 12pF -> 22pF; footprint Capacitor_SMD:C_0805_2012Metric -> PCM_JLCPCB:C_0805
- C18: footprint PCM_SparkFun-Capacitor:C_0805_2012Metric -> PCM_SparkFun-Capacitor:C_0201_0603Metric
- M1, M2, M3: value MOV-20D431K -> MOV; footprint Bourns:MOV-20D431K_Horizontal -> OpenEVSE:MOV
- moved Q3 159.2 mm to (-61.1, 39.4), turned to 0 degrees
- moved Q2 152.2 mm to (-61.1, 34.9), turned to 0 degrees
- moved D2 151.8 mm to (-41.3, 29.5)
- moved R11 149.9 mm to (-45.7, 14.6), turned to 0 degrees
- moved R41 145.7 mm to (-36.9, 23.4), turned to 0 degrees
- moved R40 143.4 mm to (-36.9, 20.5), turned to 0 degrees
- moved R31 142.9 mm to (-36.9, 17.5)
- moved R22 142.2 mm to (-41.3, 20.5), turned to 0 degrees
- moved C17 142.0 mm to (-45.4, 85.4), turned to 0 degrees
- moved L1 140.2 mm to (-49.8, 85.4), turned to 0 degrees
- moved L2 139.2 mm to (-60.7, 49.7), turned to 0 degrees
- moved C34 138.8 mm to (-27.3, 38.4), turned to 0 degrees
- moved C18 136.8 mm to (-42.2, 85.0), turned to 0 degrees
- moved R10 136.6 mm to (-45.7, 11.6)
- moved C35 136.4 mm to (-50.9, 51.9), turned to 0 degrees
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Connections:
- net Net-(C1-Pad1) renamed XGND
- R22 pad 1: ADC6 -> +5V
- R22 pad 2: +5V -> ADC6
Routing:
- net +5V: track 271.2 -> 1.33 mm, vias 9 -> 0
- net PE: track 191.4 -> 41.3 mm, vias 1 -> 0
- net AMP_READ: track 120.8 -> 5.74 mm, vias 2 -> 0
- net PP_READ: track 98.4 -> 0.00 mm, vias 4 -> 0
- net +12V: track 160.8 -> 71.5 mm, vias 2 -> 0
- net PILOT_READ: track 80.2 -> 0.00 mm, vias 4 -> 0
- net GFCI_TEST: track 78.5 -> 0.00 mm, vias 4 -> 0
- net MOSI: track 69.8 -> 0.00 mm
- net GFCI_INT: track 61.2 -> 0.00 mm, vias 2 -> 0
- net Net-(IC8-I2+): track 68.2 -> 8.97 mm, vias 2 -> 0
- net AREF: track 55.1 -> 0.00 mm, vias 2 -> 0
- net AVR_SCK: track 53.8 -> 0.00 mm, vias 2 -> 0
- net MISO: track 53.7 -> 0.00 mm
- net RESET: track 47.5 -> 0.00 mm, vias 2 -> 0
- net Net-(IC8-I1+): track 55.7 -> 8.81 mm, vias 2 -> 0
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- added copper zone on F.Cu, net XGND
- removed copper zone on B.Cu, net GND
- removed copper zone on F.Cu, net GND
- removed copper zone on B.Cu, net UGND
- removed copper zone on F.Cu, net UGND
Other:
- outline, holes or cut-outs redrawn
- board text removed: "_"

Commit message: Consolidate KiCad libraries and remove obsolete backups
Parts:
- C14: footprint OpenEVSE:C_1206_3216Metric_AC -> coreEVSE:C_1206_3216Metric_AC
- CurrentCoil1, Pilot1: footprint OpenEVSE:TerminalBlock_KF128-2.54-2P -> coreEVSE:TerminalBlock_KF128-2.54-2P
- D10, D7, D8, D9: footprint OpenEVSE:SMA_AC -> coreEVSE:SMA_AC
- D3, D4, D6: footprint OpenEVSE:SOD-123_AC -> coreEVSE:SOD-123_AC
- F1: footprint OpenEVSE:BELFUSE1A -> coreEVSE:BELFUSE1A
- FTDI1: footprint OpenEVSE:FTDI_JST_PH_1x06_P2.00mm -> coreEVSE:FTDI_JST_PH_1x06_P2.00mm
- GFCI_CT1, Pilot2: footprint OpenEVSE:TerminalBlock_KF128-2.54-4P -> coreEVSE:TerminalBlock_KF128-2.54-4P
- IC8: footprint OpenEVSE:SIL8-2 -> coreEVSE:SIL8-2
- J1: footprint OpenEVSE:AVR_ISP_2x03_P2.54mm -> coreEVSE:AVR_ISP_2x03_P2.54mm
- J4, J5, J6, J7, J8, J9: footprint OpenEVSE:Terminal_T44009_M4 -> coreEVSE:Terminal_T44009_M4
- K1, K2: footprint OpenEVSE:Relay_Hongfa_HF186F_PushIn -> coreEVSE:Relay_Hongfa_HF186F_PushIn
- L2: footprint OpenEVSE:NR5040 -> coreEVSE:NR5040
- M1, M2, M3: footprint OpenEVSE:MOV -> coreEVSE:MOV
- PS1: footprint OpenEVSE:Converter_ACDC_MeanWell_IRM-10-12_THT -> coreEVSE:Converter_ACDC_MeanWell_IRM-10-12_THT
- SH1, SH2: footprint OpenEVSE:SHORT_TOP-50 -> coreEVSE:SHORT_TOP-50
- TVS1: footprint OpenEVSE:SMB -> coreEVSE:SMB
Changed lines of the file:
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@@
 		)
 	)
-	(footprint "OpenEVSE:SOD-123_AC"
+	(footprint "coreEVSE:SOD-123_AC"
 		(layer "F.Cu")
 		(at -41.319 42.9438)
@@
 		)
 	)
-	(footprint "OpenEVSE:SOD-123_AC"
+	(footprint "coreEVSE:SOD-123_AC"
 		(layer "F.Cu")
 		(at -41.319 36.2438)
@@
 		)
 	)
-	(footprint "OpenEVSE:SMA_AC"
+	(footprint "coreEVSE:SMA_AC"
 		(layer "F.Cu")
 		(at 103.829 65.9864 -90)
@@
 		)
 	)
-	(footprint "OpenEVSE:SHORT_TOP-50"
+	(footprint "coreEVSE:SHORT_TOP-50"
 		(layer "F.Cu")
 		(at 62.3 41.8818 90)
@@
 		)
 	)
-	(footprint "OpenEVSE:SIL8-2"
+	(footprint "coreEVSE:SIL8-2"
 		(layer "F.Cu")
 		(at 95.3576 54.865)
@@
 		)
 	)
-	(footprint "OpenEVSE:NR5040"
+	(footprint "coreEVSE:NR5040"
 		(layer "F.Cu")
 		(at -60.749 49.7204)
@@
 		)
 	)
-	(footprint "OpenEVSE:SHORT_TOP-50"
+	(footprint "coreEVSE:SHORT_TOP-50"
 		(layer "F.Cu")
 		(at 56.458 31.2392)
@@
 		(embedded_fonts no)
 	)
-	(footprint "OpenEVSE:SMB"
+	(footprint "coreEVSE:SMB"
 		(layer "F.Cu")
 		(at -59.324 44.3438)
@@
 		)
 		(embedded_fonts no)
-		(model "${KIPRJMOD}/OpenEVSE.3dshapes/P6SMB16CA.step"
+		(model "${KIPRJMOD}/coreEVSE.3dshapes/P6SMB16CA.step"
 			(offset
 				(xyz 0 0 0)
@@
 		)
 	)
-	(footprint "OpenEVSE:SMA_AC"
+	(footprint "coreEVSE:SMA_AC"
 		(layer "F.Cu")
 		(at 86.43 65.7578 -90)
@@
 		(embedded_fonts no)
 	)
-	(footprint "OpenEVSE:C_1206_3216Metric_AC"
+	(footprint "coreEVSE:C_1206_3216Metric_AC"
 		(layer "F.Cu")
 		(at -41.414 46.2938)
@@
 		)
 	)
-	(footprint "OpenEVSE:SMA_AC"
+	(footprint "coreEVSE:SMA_AC"
 		(layer "F.Cu")
 		(at 98.9776 65.9864 -90)
@@
 		)
 	)
-	(footprint "OpenEVSE:SMA_AC"
+	(footprint "coreEVSE:SMA_AC"
 		(layer "F.Cu")
 		(at 91.3576 65.7324 -90)
@@
 		)
 	)
-	(footprint "OpenEVSE:SOD-123_AC"
+	(footprint "coreEVSE:SOD-123_AC"
 		(layer "F.Cu")
 		(at -41.319 32.8938)
@@
 		)
 	)
-	(footprint "OpenEVSE:TerminalBlock_KF128-2.54-2P"
+	(footprint "coreEVSE:TerminalBlock_KF128-2.54-2P"
 		(layer "B.Cu")
 		(at 24 66 90)
@@
 		)
 		(embedded_fonts no)
-		(model "${KIPRJMOD}/OpenEVSE.3dshapes/KF128-2.54-2P.wrl"
+		(model "${KIPRJMOD}/coreEVSE.3dshapes/KF128-2.54-2P.wrl"
 			(offset
 				(xyz 0 0 0)
@@
 		)
 	)
-	(footprint "OpenEVSE:TerminalBlock_KF128-2.54-4P"
+	(footprint "coreEVSE:TerminalBlock_KF128-2.54-4P"
 		(layer "B.Cu")
 		(at 24 47 90)
@@
 		)
 		(embedded_fonts no)
-		(model "${KIPRJMOD}/OpenEVSE.3dshapes/KF128-2.54-4P.wrl"
+		(model "${KIPRJMOD}/coreEVSE.3dshapes/KF128-2.54-4P.wrl"
 			(offset
 				(xyz 0 0 0)
@@
 		)
 	)
-	(footprint "OpenEVSE:Terminal_T44009_M4"
+	(footprint "coreEVSE:Terminal_T44009_M4"
 		(layer "B.Cu")
 		(at 88 110 180)
@@
 		)
 		(embedded_fonts no)
-		(model "${KIPRJMOD}/OpenEVSE.3dshapes/T44009.step"
+		(model "${KIPRJMOD}/coreEVSE.3dshapes/T44009.step"
 			(offset
 				(xyz 4.6 -5.55 -4)
@@
 		)
 	)
-	(footprint "OpenEVSE:BELFUSE1A"
+	(footprint "coreEVSE:BELFUSE1A"
 		(layer "B.Cu")
 		(at 66.17815 106.12015 90)
@@
 		)
 		(embedded_fonts no)
-		(model "${KIPRJMOD}/OpenEVSE.3dshapes/Bel_0HAAL1600-05.step"
+		(model "${KIPRJMOD}/coreEVSE.3dshapes/Bel_0HAAL1600-05.step"
 			(offset
 				(xyz 0 0 0)
@@
 		)
 	)
-	(footprint "OpenEVSE:TerminalBlock_KF128-2.54-2P"
+	(footprint "coreEVSE:TerminalBlock_KF128-2.54-2P"
 		(layer "B.Cu")
 		(at 24 35 90)
@@
 		)
 		(embedded_fonts no)
-		(model "${KIPRJMOD}/OpenEVSE.3dshapes/KF128-2.54-2P.wrl"
+		(model "${KIPRJMOD}/coreEVSE.3dshapes/KF128-2.54-2P.wrl"
 			(offset
 				(xyz 0 0 0)
@@
 		)
 	)
-	(footprint "OpenEVSE:Terminal_T44009_M4"
+	(footprint "coreEVSE:Terminal_T44009_M4"
 		(layer "B.Cu")
 		(at 28 93 180)
@@
 		)
 		(embedded_fonts no)
-		(model "${KIPRJMOD}/OpenEVSE.3dshapes/T44009.step"
+		(model "${KIPRJMOD}/coreEVSE.3dshapes/T44009.step"
 			(offset
 				(xyz 4.6 -5.55 -4)
@@
 		)
 	)
-	(footprint "OpenEVSE:AVR_ISP_2x03_P2.54mm"
+	(footprint "coreEVSE:AVR_ISP_2x03_P2.54mm"
 		(layer "B.Cu")
 		(at 115 34 180)
@@
 		)
 		(embedded_fonts no)
-		(model "${KIPRJMOD}/OpenEVSE.3dshapes/J1_AVR_ISP_2x03_P2.54mm.step"
+		(model "${KIPRJMOD}/coreEVSE.3dshapes/J1_AVR_ISP_2x03_P2.54mm.step"
 			(offset
 				(xyz -1.27 2.54 0)
@@
 		)
 	)
-	(footprint "OpenEVSE:Relay_Hongfa_HF186F_PushIn"
+	(footprint "coreEVSE:Relay_Hongfa_HF186F_PushIn"
 		(layer "B.Cu")
 		(at 105 85.5 90)
@@
 		)
 		(embedded_fonts no)
-		(model "${KIPRJMOD}/OpenEVSE.3dshapes/HF186F.step"
+		(model "${KIPRJMOD}/coreEVSE.3dshapes/HF186F.step"
 			(offset
 				(xyz -14.25 -9.25 -3.6)
@@
 		)
 	)
-	(footprint "OpenEVSE:MOV"
+	(footprint "coreEVSE:MOV"
 		(layer "B.Cu")
 		(at 41 91 -90)
@@
 		)
 		(embedded_fonts no)
-		(model "${KIPRJMOD}/OpenEVSE.3dshapes/MOV_Disc_20mm_P10mm.step"
+		(model "${KIPRJMOD}/coreEVSE.3dshapes/MOV_Disc_20mm_P10mm.step"
 			(offset
 				(xyz 0 0 0)
@@
 		)
 	)
-	(footprint "OpenEVSE:MOV"
+	(footprint "coreEVSE:MOV"
 		(layer "B.Cu")
 		(at 42 78.5 90)
@@
 		)
 		(embedded_fonts no)
-		(model "${KIPRJMOD}/OpenEVSE.3dshapes/MOV_Disc_20mm_P10mm.step"
+		(model "${KIPRJMOD}/coreEVSE.3dshapes/MOV_Disc_20mm_P10mm.step"
 			(offset
 				(xyz 0 0 0)
@@
 		)
 	)
-	(footprint "OpenEVSE:TerminalBlock_KF128-2.54-4P"
+	(footprint "coreEVSE:TerminalBlock_KF128-2.54-4P"
 		(layer "B.Cu")
 		(at 24 59 90)
@@
 		)
 		(embedded_fonts no)
-		(model "${KIPRJMOD}/OpenEVSE.3dshapes/KF128-2.54-4P.wrl"
+		(model "${KIPRJMOD}/coreEVSE.3dshapes/KF128-2.54-4P.wrl"
 			(offset
 				(xyz 0 0 0)
@@
 		)
 	)
-	(footprint "OpenEVSE:Terminal_T44009_M4"
+	(footprint "coreEVSE:Terminal_T44009_M4"
 		(layer "B.Cu")
 		(at 28 76 180)
@@
 		)
 		(embedded_fonts no)
-		(model "${KIPRJMOD}/OpenEVSE.3dshapes/T44009.step"
+		(model "${KIPRJMOD}/coreEVSE.3dshapes/T44009.step"
 			(offset
 				(xyz 4.6 -5.55 -4)
@@
 		)
 	)
-	(footprint "OpenEVSE:Terminal_T44009_M4"
+	(footprint "coreEVSE:Terminal_T44009_M4"
 		(layer "B.Cu")
 		(at 110 110 180)
@@
 		)
 		(embedded_fonts no)
-		(model "${KIPRJMOD}/OpenEVSE.3dshapes/T44009.step"
+		(model "${KIPRJMOD}/coreEVSE.3dshapes/T44009.step"
 			(offset
 				(xyz 4.6 -5.55 -4)
@@
 		)
 	)
-	(footprint "OpenEVSE:Terminal_T44009_M4"
+	(footprint "coreEVSE:Terminal_T44009_M4"
 		(layer "B.Cu")
 		(at 28 110 180)
@@
 		)
 		(embedded_fonts no)
-		(model "${KIPRJMOD}/OpenEVSE.3dshapes/T44009.step"
+		(model "${KIPRJMOD}/coreEVSE.3dshapes/T44009.step"
 			(offset
 				(xyz 4.6 -5.55 -4)
@@
 		)
 	)
-	(footprint "OpenEVSE:Terminal_T44009_M4"
+	(footprint "coreEVSE:Terminal_T44009_M4"
 		(layer "B.Cu")
 		(at 50 110 180)
@@
 		)
 		(embedded_fonts no)
-		(model "${KIPRJMOD}/OpenEVSE.3dshapes/T44009.step"
+		(model "${KIPRJMOD}/coreEVSE.3dshapes/T44009.step"
 			(offset
 				(xyz 4.6 -5.55 -4)
@@
 		)
 	)
-	(footprint "OpenEVSE:Relay_Hongfa_HF186F_PushIn"
+	(footprint "coreEVSE:Relay_Hongfa_HF186F_PushIn"
 		(layer "B.Cu")
 		(at 83 85.5 90)
@@
 		)
 		(embedded_fonts no)
-		(model "${KIPRJMOD}/OpenEVSE.3dshapes/HF186F.step"
+		(model "${KIPRJMOD}/coreEVSE.3dshapes/HF186F.step"
 			(offset
 				(xyz -14.25 -9.25 -3.6)
@@
 		)
 	)
-	(footprint "OpenEVSE:FTDI_JST_PH_1x06_P2.00mm"
+	(footprint "coreEVSE:FTDI_JST_PH_1x06_P2.00mm"
 		(layer "B.Cu")
 		(at 116 48 -90)
@@
 		)
 		(embedded_fonts no)
-		(model "${KIPRJMOD}/OpenEVSE.3dshapes/FTDI_JST_PH_1x06_P2.00mm.step"
+		(model "${KIPRJMOD}/coreEVSE.3dshapes/FTDI_JST_PH_1x06_P2.00mm.step"
 			(offset
 				(xyz -5 -0.28 0)
@@
 		)
 	)
-	(footprint "OpenEVSE:MOV"
+	(footprint "coreEVSE:MOV"
 		(layer "B.Cu")
 		(at 37 89.2528 90)
@@
 		)
 		(embedded_fonts no)
-		(model "${KIPRJMOD}/OpenEVSE.3dshapes/MOV_Disc_20mm_P10mm.step"
+		(model "${KIPRJMOD}/coreEVSE.3dshapes/MOV_Disc_20mm_P10mm.step"
 			(offset
 				(xyz 0 0 0)
@@
 		)
 	)
-	(footprint "OpenEVSE:Converter_ACDC_MeanWell_IRM-10-12_THT"
+	(footprint "coreEVSE:Converter_ACDC_MeanWell_IRM-10-12_THT"
 		(layer "B.Cu")
 		(at 60 97 90)
@@
 		)
 		(embedded_fonts no)
-		(model "${KIPRJMOD}/OpenEVSE.3dshapes/MeanWell_IRM-10-12.step"
+		(model "${KIPRJMOD}/coreEVSE.3dshapes/MeanWell_IRM-10-12.step"
 			(offset
 				(xyz 0 0 0)

Commit message: end
Parts:
- moved Q3 177.2 mm to (115.6, 52.3), turned to -90 degrees
- moved Q2 172.4 mm to (110.4, 52.3), turned to -90 degrees
- moved R11 165.7 mm to (116.6, 48.0), turned to -90 degrees
- moved R24 154.1 mm to (111.3, 48.0), turned to 90 degrees
- moved D2 152.8 mm to (105.1, 73.2)
- moved R40 139.3 mm to (101.9, 31.5), turned to 180 degrees
- moved R41 138.9 mm to (101.9, 28.9)
- moved D5 129.0 mm to (83.2, 73.2)
- moved C34 126.0 mm to (98.4, 29.8), turned to -90 degrees
- moved L2 114.5 mm to (53.4, 41.3), turned to 180 degrees
- moved U1 111.5 mm to (56.0, 46.2)
- moved C24 103.7 mm to (53.9, 52.6), turned to 180 degrees
- moved C23 102.1 mm to (53.8, 55.5), turned to 180 degrees
- moved C28 99.7 mm to (55.8, 49.5), turned to 180 degrees
- moved C29 97.8 mm to (52.0, 46.1), turned to -90 degrees
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Routing:
- net +5V: track 1.33 -> 99.9 mm, vias 0 -> 1
- net Net-(D7-PadA): track 0.00 -> 80.6 mm, vias 0 -> 2
- net MISO: track 0.00 -> 52.4 mm, vias 0 -> 1
- net MOSI: track 0.00 -> 50.8 mm, vias 0 -> 1
- net DC_RELAY_2: track 0.00 -> 50.8 mm, vias 0 -> 2
- net GFCI_TEST: track 0.00 -> 49.0 mm, vias 0 -> 2
- net DC_RELAY_1: track 0.00 -> 46.6 mm, vias 0 -> 2
- net DC_RELAY_C1: track 0.20 -> 42.5 mm
- net Net-(D8-PadA): track 0.00 -> 40.1 mm, vias 0 -> 2
- net Net-(D9-PadA): track 29.2 -> 66.9 mm
- net DC_RELAY_C2: track 0.36 -> 26.0 mm
- net Net-(D10-PadA): track 21.7 -> 39.3 mm
- net Net-(IC3B-+IN2): track 0.00 -> 17.1 mm
- net Net-(IC3A--IN1): track 0.00 -> 16.9 mm, vias 0 -> 2
- net +12V: track 71.5 -> 86.7 mm
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- added copper zone on F.Cu, net GND
Other:
- outline, holes or cut-outs redrawn

Commit message: fix
Parts:
- moved C15 115.9 mm to (-9.66, -26.1), turned to 90 degrees
- moved TVS1 98.4 mm to (8.34, -27.1), turned to 180 degrees
- moved R6 85.1 mm to (17.9, -30.6), turned to 180 degrees
- moved R3 80.7 mm to (27.8, 35.4), turned to 180 degrees
- moved R2 80.7 mm to (27.8, 32.4)
- moved D6 74.9 mm to (32.8, 32.4)
- moved C6 72.4 mm to (10.3, -17.1), turned to -90 degrees
- moved C5 72.3 mm to (-7.66, -31.1), turned to -90 degrees
- moved R7 71.8 mm to (0.42, -27.6), turned to 180 degrees
- moved C13 70.9 mm to (6.84, -21.1), turned to 90 degrees
- moved C10 62.7 mm to (6.84, -17.1), turned to -90 degrees
- moved R5 58.3 mm to (-13.2, -27.6), turned to 90 degrees
- moved C26 56.5 mm to (-5.16, -19.6), turned to 90 degrees
- moved R1 55.6 mm to (-6.66, -26.1), turned to 90 degrees
- moved FTDI1 52.8 mm to (85.3, 23.9), turned to 0 degrees
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Routing:
- net +5V: track 99.9 -> 120.1 mm
- net PP: track 0.00 -> 17.5 mm
- net PILOT: track 0.00 -> 7.02 mm
- net Net-(IC1-Pad1): track 0.00 -> 3.55 mm
- net Net-(IC1A--): track 0.00 -> 2.55 mm
- net PP_READ: track 0.00 -> 2.44 mm

Commit message: fix PCB
Parts:
- C28: footprint PCM_SparkFun-Capacitor:C_0805_2012Metric -> PCM_JLCPCB:C_0805
- moved C12 180.0 mm to (130.0, 88.5)
- moved C17 180.0 mm to (134.4, 94.2)
- moved C18 180.0 mm to (137.6, 93.9)
- moved C19 180.0 mm to (134.4, 79.4)
- moved C20 180.0 mm to (134.4, 82.5)
- moved C21 180.0 mm to (134.4, 85.5)
- moved C27 180.0 mm to (138.9, 79.4)
- moved C3 180.0 mm to (130.0, 79.4)
- moved C35 180.0 mm to (128.9, 60.7)
- moved C4 180.0 mm to (130.0, 82.5)
- moved C9 180.0 mm to (130.0, 85.5)
- moved L1 180.0 mm to (130.0, 94.3)
- moved R10 178.2 mm to (130.1, 45.0)
- moved R14 178.2 mm to (130.1, 50.9)
- moved R22 178.2 mm to (134.5, 53.9)
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Routing:
- net +5V: track 120.1 -> 199.0 mm
- net +12V: track 86.7 -> 115.3 mm
- net PILOT_READ: track 0.00 -> 23.3 mm
- net PILOT: track 7.02 -> 16.2 mm
- net Net-(IC1C-V-): track 0.00 -> 8.73 mm
- net Net-(IC1A--): track 2.55 -> 7.55 mm
- net Net-(U2-CAP+): track 0.00 -> 3.19 mm
- net Net-(U2-CAP-): track 0.00 -> 3.17 mm
- net UGND: track 12.7 -> 14.9 mm
- net Net-(IC1B--): track 0.00 -> 1.27 mm
