File: evse.kicad_pcb (KiCad board)
At the start: 2 copper layers, 100 x 100 mm, 119 parts, among them IC1 LF353, IC3 LM358, IC8 HCPL-2731S, J1 ISP, J4 T44009, J5 T44009, J6 T44009, J7 T44009, J8 T44009, J9 T44009, K1 HF186F/12-HCTF, K2 HF186F/12-HCTF, M1 MOV, M2 MOV, M3 MOV, Q2 MMBT2222A, Q3 MMBT2222A, U1 AP63205WU, U2 TC1044S, U3 MCP9808, U4 ATmega328P-AU, Y1 16MHz

Commit message: night
Parts:
- moved R14 81.5 mm to (48.6, 50.8), turned to 90 degrees
- moved C27 79.2 mm to (76.6, 30.5)
- moved R31 61.3 mm to (77.6, 52.3)
- moved R10 60.9 mm to (70.0, 34.9)
- moved C3 53.4 mm to (97.2, 37.4), turned to 90 degrees
- moved R22 49.7 mm to (85.7, 44.3), turned to 180 degrees
- moved R27 49.5 mm to (90.1, 40.0), turned to 180 degrees
- moved C35 48.9 mm to (84.8, 39.6), turned to 90 degrees
- moved SH1 8.36 mm to (87.9, 36.9)
- moved SH2 5.34 mm to (67.9, 42.0)
- moved U4 5.33 mm to (78.0, 39.5)
- moved C1 5.23 mm to (70.6, 38.6)
- moved C2 5.23 mm to (70.6, 45.0)
- moved Y1 5.23 mm to (70.7, 41.9)
- moved C33 0.80 mm to (48.6, 46.2)
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Routing:
- net VCC: track 4.77 -> 19.9 mm, vias 2 -> 3
- net MOSI: track 50.8 -> 43.9 mm
- net UGND: track 14.9 -> 21.4 mm
- net DC_RELAY_1: track 46.6 -> 41.1 mm
- net +5V: track 199.0 -> 204.4 mm
- net MISO: track 52.4 -> 47.2 mm
- net PILOT_READ: track 23.3 -> 28.3 mm
- net GFCI_TEST: track 49.0 -> 54.0 mm
- net DC_RELAY_2: track 50.8 -> 46.4 mm
- net Net-(IC3A-OUT1): track 4.42 -> 7.51 mm
- net Net-(IC3B--IN2): track 9.40 -> 12.5 mm

Commit message: final
Parts:
- moved C18 76.7 mm to (89.5, 34.1)
- moved C12 73.0 mm to (85.6, 30.4), turned to 180 degrees
- moved C17 71.6 mm to (90.0, 38.0)
- moved C20 69.4 mm to (85.7, 33.0)
- moved C21 68.9 mm to (91.9, 31.2), turned to 180 degrees
- moved L1 67.4 mm to (93.7, 37.5), turned to -90 degrees
- moved C19 62.2 mm to (90.1, 35.8)
- moved C9 53.3 mm to (107.1, 37.4), turned to 90 degrees
- moved C4 52.2 mm to (103.7, 37.4), turned to 90 degrees
- moved SH1 8.59 mm to (87.3, 28.4)
- moved R31 7.13 mm to (70.9, 50.0)
- moved R22 3.05 mm to (88.6, 45.2), turned to 90 degrees
- moved C27 0.10 mm to (76.6, 30.4)
Routing:
- net UGND: track 21.4 -> 29.2 mm
- net ADC6: track 0.00 -> 7.83 mm
- net VCC: track 19.9 -> 24.2 mm
- net Net-(L1-Pad2): track 0.00 -> 3.93 mm
- net PILOT_READ: track 28.3 -> 25.9 mm
- net +5V: track 204.4 -> 206.1 mm

Commit message: fix Y1
Parts:
- C1, C2: value 22pF -> 12pF; footprint PCM_JLCPCB:C_0805 -> Capacitor_SMD:C_0402_1005Metric
- Y1: value 16MHz -> FA-238A 16MHz CL=8pF; footprint PCM_SparkFun-Clock:Crystal_SMD_3.2x2.5mm -> Crystal:Crystal_SMD_SeikoEpson_TSX3225-4Pin_3.2x2.5mm
- moved C1 1.04 mm to (69.6, 38.8), turned to -90 degrees
- moved SH2 0.93 mm to (67.1, 41.6), turned to 180 degrees
- moved C2 0.62 mm to (71.2, 45.1), turned to 90 degrees
- moved Y1 0.33 mm to (70.4, 41.9)
Connections:
- Y1 pad 2: Net-(U4-XTAL1/PB6) -> XGND
- Y1 pad 3: unconnected-(Y1-NC1-Pad3) -> Net-(U4-XTAL1/PB6)
- Y1 pad 4: unconnected-(Y1-NC2-Pad4) -> XGND
Routing:
- net Net-(U4-XTAL1/PB6): track 4.93 -> 0.00 mm
- net Net-(U4-XTAL2/PB7): track 4.85 -> 0.03 mm

Commit message: fix SH3
Parts:
- added SH3: NetTie_2, NetTie:NetTie-2_SMD_Pad0.5mm, F.Cu at (22.0, 41.9)
- SH1, SH2: footprint coreEVSE:SHORT_TOP-50 -> NetTie:NetTie-2_SMD_Pad0.5mm
Changed lines of the file:
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@@
 		)
 	)
-	(footprint "coreEVSE:SHORT_TOP-50"
+	(footprint "NetTie:NetTie-2_SMD_Pad0.5mm"
 		(layer "F.Cu")
 		(at 67.1006 41.5516 180)
-		(descr "OpenEVSE soldered top-layer short, original Eagle SHORT_TOP-50")
+		(descr "Net tie, 2 pin, 0.5mm square SMD pads")
+		(tags "net tie")
 		(property "Reference" "SH2"
-			(at -0.3302 -3.2004 0)
+			(at 0 -1.2 180)
 			(layer "F.SilkS")
+			(hide yes)
 			(effects
 				(font
@@
 		)
 		(property "Value" "NetTie_2"
-			(at 0 2.032 0)
+			(at 0 1.2 180)
 			(layer "F.Fab")
 			(hide yes)
@@
 		)
 		(property "Datasheet" ""
-			(at 0 0 0)
+			(at 0 0 180)
+			(unlocked yes)
 			(layer "F.Fab")
 			(hide yes)
@@
 				(font
 					(size 1.27 1.27)
+					(thickness 0.15)
 				)
 			)
 		)
 		(property "Description" "Net tie, 2 pins"
-			(at 0 0 0)
+			(at 0 0 180)
+			(unlocked yes)
 			(layer "F.Fab")
 			(hide yes)
@@
 				(font
 					(size 1.27 1.27)
+					(thickness 0.15)
 				)
 			)
@@
 			)
 		)
-		(attr exclude_from_bom)
+		(attr exclude_from_bom allow_missing_courtyard)
+		(net_tie_pad_groups "1, 2")
 		(duplicate_pad_numbers_are_jumpers no)
-		(fp_line
-			(start -1.27 0.635)
-			(end 1.27 0.635)
-			(stroke
-				(width 0.15)
-				(type default)
+		(fp_poly
+			(pts
+				(xy -0.5 -0.25) (xy 0.5 -0.25) (xy 0.5 0.25) (xy -0.5 0.25)
 			)
-			(layer "F.SilkS")
-		)
-		(fp_line
-			(start -1.27 -0.635)
-			(end 1.27 -0.635)
 			(stroke
-				(width 0.15)
-				(type default)
+				(width 0)
+				(type solid)
 			)
-			(layer "F.SilkS")
+			(fill yes)
+			(layer "F.Cu")
 		)
-		(pad "1" smd rect
-			(at 0.635 0 180)
-			(size 1.27 1.27)
+		(pad "1" smd circle
+			(at -0.5 0 180)
+			(size 0.5 0.5)
 			(layers "F.Cu")
 			(net "UGND")
@@
 			(pintype "passive")
 		)
-		(pad "2" smd rect
-			(at -0.635 0 180)
-			(size 1.27 1.27)
+		(pad "2" smd circle
+			(at 0.5 0 180)
+			(size 0.5 0.5)
 			(layers "F.Cu")
 			(net "XGND")
@@
 		)
 	)
-	(footprint "coreEVSE:SHORT_TOP-50"
+	(footprint "NetTie:NetTie-2_SMD_Pad0.5mm"
 		(layer "F.Cu")
 		(at 87.319 28.369)
-		(descr "OpenEVSE soldered top-layer short, original Eagle SHORT_TOP-50")
+		(descr "Net tie, 2 pin, 0.5mm square SMD pads")
+		(tags "net tie")
 		(property "Reference" "SH1"
-			(at 3.035 -2.05 0)
+			(at 0 -1.2 0)
 			(layer "F.SilkS")
+			(hide yes)
 			(effects
 				(font
@@
 		)
 		(property "Value" "NetTie_2"
-			(at 0 2.032 0)
+			(at 0 1.2 0)
 			(layer "F.Fab")
 			(hide yes)
@@
 		(property "Datasheet" ""
 			(at 0 0 0)
+			(unlocked yes)
 			(layer "F.Fab")
 			(hide yes)
@@
 				(font
 					(size 1.27 1.27)
+					(thickness 0.15)
 				)
 			)
@@
 		(property "Description" "Net tie, 2 pins"
 			(at 0 0 0)
+			(unlocked yes)
 			(layer "F.Fab")
 			(hide yes)
@@
 				(font
 					(size 1.27 1.27)
+					(thickness 0.15)
 				)
 			)
@@
 			)
 		)
-		(attr exclude_from_bom)
+		(attr exclude_from_bom allow_missing_courtyard)
+		(net_tie_pad_groups "1, 2")
 		(duplicate_pad_numbers_are_jumpers no)
-		(fp_line
-			(start -1.27 -0.635)
-			(end 1.27 -0.635)
-			(stroke
-				(width 0.15)
-				(type default)
+		(fp_poly
+			(pts
+				(xy -0.5 -0.25) (xy 0.5 -0.25) (xy 0.5 0.25) (xy -0.5 0.25)
 			)
-			(layer "F.SilkS")
-		)
-		(fp_line
-			(start -1.27 0.635)
-			(end 1.27 0.635)
 			(stroke
-				(width 0.15)
-				(type default)
+				(width 0)
+				(type solid)
 			)
-			(layer "F.SilkS")
+			(fill yes)
+			(layer "F.Cu")
 		)
-		(pad "1" smd rect
-			(at 0.635 0)
-			(size 1.27 1.27)
+		(pad "1" smd circle
+			(at -0.5 0)
+			(size 0.5 0.5)
 			(layers "F.Cu")
 			(net "GND")
@@
 			(pintype "passive")
 		)
-		(pad "2" smd rect
-			(at -0.635 0)
-			(size 1.27 1.27)
+		(pad "2" smd circle
+			(at 0.5 0)
+			(size 0.5 0.5)
 			(layers "F.Cu")
 			(net "UGND")
@@
 		)
 	)
+	(footprint "NetTie:NetTie-2_SMD_Pad0.5mm"
+		(layer "F.Cu")
+		(at 21.9528 41.9286)
+		(descr "Net tie, 2 pin, 0.5mm square SMD pads")
+		(tags "net tie")
+		(property "Reference" "SH3"
+			(at 0 -1.2 0)
+			(layer "F.SilkS")
+			(hide yes)
+			(effects
+				(font
+					(size 1 1)
+					(thickness 0.15)
+				)
+			)
+		)
+		(property "Value" "NetTie_2"
+			(at 0 1.2 0)
+			(layer "F.Fab")
+			(hide yes)
+			(effects
+				(font
+					(size 1 1)
+					(thickness 0.15)
+				)
+			)
+		)
+		(property "Datasheet" ""
+			(at 0 0 0)
+			(unlocked yes)
+			(layer "F.Fab")
+			(hide yes)
+			(effects
+				(font
+					(size 1.27 1.27)
+					(thickness 0.15)
+				)
+			)
+		)
+		(property "Description" "Single-point PE to electronics GND reference bond for Control Pilot"
+			(at 0 0 0)
+			(unlocked yes)
+			(layer "F.Fab")
+			(hide yes)
+			(effects
+				(font
+					(size 1.27 1.27)
+					(thickness 0.15)
+				)
+			)
+		)
+		(property ki_fp_filters "Net*Tie*")
+		(sheetname "/")
+		(sheetfile "evse.kicad_sch")
+		(units
+			(unit
+				(name "A")
+				(pins "1" "2")
+			)
+		)
+		(attr exclude_from_bom allow_missing_courtyard)
+		(net_tie_pad_groups "1, 2")
+		(duplicate_pad_numbers_are_jumpers no)
+		(fp_poly
+			(pts
+				(xy -0.5 -0.25) (xy 0.5 -0.25) (xy 0.5 0.25) (xy -0.5 0.25)
+			)
+			(stroke
+				(width 0)
+				(type solid)
+			)
+			(fill yes)
+			(layer "F.Cu")
+		)
+		(pad "1" smd circle
+			(at -0.5 0)
+			(size 0.5 0.5)
+			(layers "F.Cu")
+			(net "GND")
+			(pinfunction "1_1")
+			(pintype "passive")
+		)
+		(pad "2" smd circle
+			(at 0.5 0)
+			(size 0.5 0.5)
+			(layers "F.Cu")
+			(net "PE")
+			(pinfunction "2_2")
+			(pintype "passive")
+		)
+		(embedded_fonts no)
+	)
 	(footprint "Resistor_SMD:R_0805_2012Metric"

Commit message: done
Parts:
- removed U$3, U$9: HOLE, coreEVSE:HOLE
- added R42: 47k, Resistor_SMD:R_0805_2012Metric, F.Cu at (67.3, 52.4)
- added R43: 47k, Resistor_SMD:R_0805_2012Metric, F.Cu at (77.3, 52.4)
- added UNK_HOLE_1: , dummyfp1, F.Cu at (23.0, 23.0)
- added UNK_HOLE_1: , dummyfp1, F.Cu at (117.0, 23.0)
- C10, C13, C26, C5, C6: footprint Capacitor_SMD:C_0805_2012Metric -> Capacitor_SMD:C_1210_3225Metric
- D10, D7, D8, D9: value 1N4004 -> S1M
- R32, R33, R34, R35, R36, R37, R38, R39: footprint Resistor_SMD:R_1210_3225Metric -> Resistor_SMD:R_2512_6332Metric
- moved R34 44.0 mm to (69.0, 60.4)
- moved R24 41.5 mm to (69.9, 50.4)
- moved R35 37.2 mm to (69.0, 65.4), turned to 0 degrees
- moved Q2 37.1 mm to (73.3, 52.4), turned to 0 degrees
- moved R11 36.8 mm to (79.8, 50.4)
- moved Q3 32.4 mm to (83.3, 52.4), turned to 0 degrees
- moved R32 29.3 mm to (87.8, 60.4), turned to 0 degrees
- moved R38 29.0 mm to (114.3, 60.4), turned to 0 degrees
- moved R37 28.4 mm to (96.3, 65.4), turned to 0 degrees
- moved R39 28.3 mm to (114.3, 65.4)
- moved R36 28.0 mm to (96.3, 60.4), turned to 180 degrees
- moved R33 26.8 mm to (87.8, 65.4)
- moved R10 16.0 mm to (84.3, 27.7), turned to -90 degrees
- moved R31 15.4 mm to (85.3, 44.4)
- moved SH1 13.5 mm to (73.8, 28.9), turned to -90 degrees
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Connections:
- U3 pad 5: unconnected-(U3-A2-Pad5) -> GND
- U3 pad 6: unconnected-(U3-A1-Pad6) -> GND
- U3 pad 7: unconnected-(U3-A0-Pad7) -> GND
Routing:
- net Net-(D7-PadA): track 80.6 -> 4.25 mm, vias 2 -> 0
- net Net-(D9-PadA): track 66.9 -> 3.42 mm, vias 2 -> 0
- net +12V: track 115.3 -> 173.2 mm, vias 0 -> 2
- net +5V: track 206.1 -> 259.9 mm
- net PILOT: track 16.2 -> 63.2 mm, vias 0 -> 2
- net AVR_SCK: track 0.00 -> 39.2 mm, vias 0 -> 1
- net DC_RELAY_2: track 46.4 -> 9.31 mm, vias 2 -> 0
- net AC_N_OUT: track 0.00 -> 36.7 mm
- net Net-(D8-PadA): track 40.1 -> 3.84 mm, vias 2 -> 0
- net Net-(D10-PadA): track 39.3 -> 3.81 mm, vias 2 -> 0
- net SCL: track 7.93 -> 38.6 mm, vias 1 -> 2
- net DC_RELAY_1: track 41.1 -> 10.4 mm, vias 2 -> 0
- net SDA: track 10.6 -> 41.2 mm, vias 1 -> 3
- net RESET: track 0.00 -> 30.2 mm, vias 0 -> 2
- net UGND: track 29.2 -> 0.00 mm
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- added copper zone on B.Cu, net GND
- added copper zone on F.Cu, net UGND

Commit message: tested
Parts:
- removed SH3: NetTie_2, NetTie:NetTie-2_SMD_Pad0.5mm
- C21: footprint PCM_SparkFun-Capacitor:C_0805_2012Metric -> PCM_JLCPCB:C_0805
- U2: value TC1044S -> LTC1144IS8#TRPBF
- moved F1 9.33 mm to (57.9, 101.7), turned to -90 degrees
- moved C4 9.05 mm to (115.7, 34.5), turned to 0 degrees
- moved D3 8.16 mm to (35.2, 43.9), turned to 180 degrees
- moved R25 6.17 mm to (39.3, 61.9), turned to -90 degrees
- moved C9 5.12 mm to (115.7, 37.8), turned to 0 degrees
- moved C11 3.93 mm to (34.3, 61.9), turned to -90 degrees
- moved R21 3.59 mm to (36.8, 61.9), turned to 90 degrees
- moved R20 3.05 mm to (31.0, 55.1)
- moved C7 2.76 mm to (34.8, 52.4)
- moved R16 2.75 mm to (34.7, 55.0)
- moved R23 2.74 mm to (27.2, 56.4)
- moved R18 2.60 mm to (35.9, 46.4)
- moved R1 2.57 mm to (65.1, 28.7), turned to 0 degrees
- moved R5 2.55 mm to (75.6, 29.6)
- moved D6 2.50 mm to (29.4, 28.9), turned to 90 degrees
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Connections:
- F1 pad 1: ACNIN -> ACLIN
- F1 pad 2: Net-(PS1-AC/N) -> Net-(PS1-AC/L)
- PS1 pad 1: Net-(PS1-AC/N) -> ACNIN
- PS1 pad 2: ACLIN -> Net-(PS1-AC/L)
Routing:
- net AMP_READ: track 5.75 -> 77.4 mm, vias 0 -> 1
- net PE: track 42.9 -> 112.2 mm, vias 0 -> 1
- net PP_READ: track 3.05 -> 65.0 mm, vias 0 -> 2
- net PILOT: track 63.2 -> 11.4 mm, vias 2 -> 0
- net GFCI_INT: track 1.94 -> 42.2 mm, vias 0 -> 2
- net RESET: track 30.2 -> 70.3 mm, vias 2 -> 4
- net Net-(IC1-Pad1): track 3.55 -> 36.2 mm, vias 0 -> 1
- net PWM: track 0.00 -> 29.1 mm, vias 0 -> 2
- net WELD_DETECT: track 0.00 -> 25.1 mm, vias 0 -> 2
- net GMI_LINE: track 0.00 -> 22.2 mm, vias 0 -> 2
- net VCC: track 15.3 -> 32.4 mm, vias 0 -> 2
- net Net-(PS1-AC/L): track 0.00 -> 13.1 mm
- net Net-(PS1-AC/N): track 10.9 -> 0.00 mm
- net +12V: track 173.2 -> 183.1 mm
- net +5V: track 259.9 -> 250.2 mm
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- removed copper zone on B.Cu, net GND

Commit message: new
Parts:
- added SH3: NetTie_2, NetTie:NetTie-2_SMD_Pad0.5mm, F.Cu at (0.75, 0.25)
- L2: footprint coreEVSE:NR5040 -> Inductor_SMD:L_Bourns_SRP5030T
- moved F1 5.06 mm to (63.0, 101.5)
- moved C32 0.50 mm to (58.8, 41.3)
Routing:
- net +5V: track 250.2 -> 260.8 mm
- net ACLIN: track 7.48 -> 0.00 mm, vias 1 -> 0
- net Net-(PS1-AC/L): track 13.1 -> 18.2 mm
- net Net-(U1-SW): track 9.40 -> 10.4 mm

Commit message: fix
Parts:
- removed FID2, FID3, FID4: FIDUCIAL1X2, Fiducial:Fiducial_1mm_Mask2mm
- removed SH3: NetTie_2, NetTie:NetTie-2_SMD_Pad0.5mm
- C12, C15, C19, C20, C23, C24, C27, C29, C3, C33, C4, C9: footprint PCM_SparkFun-Capacitor:C_0805_2012Metric -> Capacitor_SMD:C_0805_2012Metric
- C21, C28: footprint PCM_JLCPCB:C_0805 -> Capacitor_SMD:C_0805_2012Metric
- D2, D5: value SS14 -> B5819W
- K1, K2: value HF186F/12-HCTF -> HF186F/12-HTF
- L1: footprint PCM_SparkFun-Coil:0805 -> Inductor_SMD:L_0805_2012Metric
- Q2, Q3: value MMBT2222A -> AO3400A
- moved TVS1 42.0 mm to (27.5, 32.8)
- moved SH1 10.9 mm to (84.3, 31.9)
- moved R3 5.51 mm to (32.5, 32.5)
- moved R2 5.13 mm to (23.0, 28.2), turned to 0 degrees
- moved D6 2.82 mm to (31.0, 26.6)
- moved C18 2.55 mm to (88.8, 31.4), turned to 180 degrees
- moved C21 2.23 mm to (91.8, 33.4)
- moved C35 1.19 mm to (88.7, 33.7), turned to 180 degrees
- moved FID1 0.71 mm to (26.0, 26.0)
- moved R31 0.44 mm to (85.3, 44.0)
Routing:
- net Net-(IC1-Pad1): track 36.2 -> 16.8 mm
- net PP: track 17.5 -> 28.2 mm
- net +5V: track 260.8 -> 253.9 mm
- net VCC: track 32.4 -> 27.6 mm
- net PP_READ: track 65.0 -> 68.7 mm
