File: evse.kicad_sch (KiCad schematic)
At the start: 111 parts, among them IC1 LF353, IC2 ATmega328P, IC3 LM358, IC8 HCPL-2731S, J1 ISP, J4 T44009, J5 T44009, J6 T44009, J7 T44009, J8 T44009, J9 T44009, K1 HF186F/12-HCTF, K2 HF186F/12-HCTF, M1 MOV, M2 MOV, M3 MOV, Q2 MMBT2222A, Q3 MMBT2222A, U1 AP63205WU, U2 TC1044S, U3 MCP9808, Y1 16MHz

Commit message: fix
Parts:
- removed IC2: ATmega328P, PCM_SparkFun-Semiconductor-Standard:TQFP-32_7x7mm_P0.8mm, symbol PCM_SparkFun-IC-Microcontroller:ATmega328P-AU
- added FID1, FID2, FID3, FID4: FIDUCIAL1X2, Fiducial:Fiducial_1mm_Mask2mm, symbol OpenEVSE_PLUS_v6.5.1-eagle-import:FIDUCIAL1X2.5
- added U$3, U$9: HOLE, coreEVSE:HOLE, symbol OpenEVSE_PLUS_v6.5.1-eagle-import:HOLE
- added U4: ATmega328P-AU, PCM_JLCPCB:TQFP-32_7x7mm_P0.8mm, symbol PCM_JLCPCB-MCUs:ATmega328P-AU
- C1, C2: value 12pF -> 22pF; footprint Capacitor_SMD:C_0805_2012Metric -> PCM_JLCPCB:C_0805
- C18: footprint PCM_SparkFun-Capacitor:C_0805_2012Metric -> PCM_SparkFun-Capacitor:C_0201_0603Metric
Connections:
- net +5V: now also R22.1, U4.18 (AVCC); no longer R22.2
- net ADC6: now also R22.2, U4.19 (ADC6); no longer R22.1
- net AMP_READ: now also U4.23 (PC0)
- net AREF: now also U4.20 (AREF)
- net AVR_SCK: now also U4.17 (PB5)
- net DC_RELAY_1: now also U4.9 (PD5)
- net DC_RELAY_2: now also U4.10 (PD6)
- net GFCI_INT: now also U4.32 (PD2)
- net GFCI_TEST: now also U4.12 (PB0)
- net GMI_LINE: now also U4.2 (PD4)
- net GND: now also U$9.P$1 (GND)
- net MISO: now also U4.16 (PB4)
- net MOSI: now also U4.15 (PB3)
- net PE: now also U$3.P$1 (GND)
- net PILOT_READ: now also U4.24 (PC1)
- net PP_READ: now also U4.25 (PC2)
- net PWM: now also U4.14 (PB2)
- net RESET: now also U4.29 (~{RESET}/PC6)
- net RX-I: now also U4.30 (PD0)
- net SCL: now also U4.28 (PC5)
- net SDA: now also U4.27 (PC4)
- net TX: now also U4.31 (PD1)
- net UGND: now also U4.21 (GND), U4.3 (GND), U4.5 (GND)
- net VCC: now also U4.4 (VCC), U4.6 (VCC)
- net WELD_DETECT: now also U4.1 (PD3)
- net at R31.1: now also U4.11 (PD7)
- net at C1.2, Y1.2: now also U4.7 (XTAL1/PB6)
- net at C2.2, Y1.1: now also U4.8 (XTAL2/PB7)
- net XGND: now reaches C1.1, C2.1, SH2.2
Other:
- moved on the sheet: C1, C12, C2, C20, C21, Pilot1, Pilot2, R22, R31, SH1, SH2, Y1

Commit message: Consolidate KiCad libraries and remove obsolete backups
Parts:
- C11, C16, C34, C7: symbol GFI_Original:SparkFun_CAP0805 -> coreEVSE:SparkFun_CAP0805
- C14: footprint OpenEVSE:C_1206_3216Metric_AC -> coreEVSE:C_1206_3216Metric_AC; symbol GFI_Original:SparkFun_CAP_POL1206 -> coreEVSE:SparkFun_CAP_POL1206
- CurrentCoil1, Pilot1: footprint OpenEVSE:TerminalBlock_KF128-2.54-2P -> coreEVSE:TerminalBlock_KF128-2.54-2P; symbol OpenEVSE:KF128-2.54-2P -> coreEVSE:KF128-2.54-2P
- D1, D11: symbol GFI_Original:diode_BAS40-06 -> coreEVSE:diode_BAS40-06
- D10, D7, D8, D9: footprint OpenEVSE:SMA_AC -> coreEVSE:SMA_AC; symbol ACTEST_Original:diode_MBRA340T3 -> coreEVSE:diode_MBRA340T3
- D3, D4, D6: footprint OpenEVSE:SOD-123_AC -> coreEVSE:SOD-123_AC; symbol GFI_Original:diode_DIODE-SOD123 -> coreEVSE:diode_DIODE-SOD123
- F1: footprint OpenEVSE:BELFUSE1A -> coreEVSE:BELFUSE1A
- FTDI1: footprint OpenEVSE:FTDI_JST_PH_1x06_P2.00mm -> coreEVSE:FTDI_JST_PH_1x06_P2.00mm
- GFCI_CT1, Pilot2: footprint OpenEVSE:TerminalBlock_KF128-2.54-4P -> coreEVSE:TerminalBlock_KF128-2.54-4P; symbol OpenEVSE:KF128-2.54-4P -> coreEVSE:KF128-2.54-4P
- IC3: symbol GFI_Original:SparkFun_LMV358 -> coreEVSE:SparkFun_LMV358
- IC8: footprint OpenEVSE:SIL8-2 -> coreEVSE:SIL8-2; symbol ACTEST_Original:OpenEVSE_HCPL-2731S -> coreEVSE:OpenEVSE_HCPL-2731S
- J1: footprint OpenEVSE:AVR_ISP_2x03_P2.54mm -> coreEVSE:AVR_ISP_2x03_P2.54mm
- J4, J5, J6, J7, J8, J9: footprint OpenEVSE:Terminal_T44009_M4 -> coreEVSE:Terminal_T44009_M4; symbol OpenEVSE:T44009 -> coreEVSE:T44009
- K1, K2: footprint OpenEVSE:Relay_Hongfa_HF186F_PushIn -> coreEVSE:Relay_Hongfa_HF186F_PushIn; symbol OpenEVSE:HF186F -> coreEVSE:HF186F
- L2: footprint OpenEVSE:NR5040 -> coreEVSE:NR5040
- M1, M2, M3: footprint OpenEVSE:MOV -> coreEVSE:MOV; symbol MOV_Original:OpenEVSE_MOV -> coreEVSE:OpenEVSE_MOV
- PS1: footprint OpenEVSE:Converter_ACDC_MeanWell_IRM-10-12_THT -> coreEVSE:Converter_ACDC_MeanWell_IRM-10-12_THT
- R14, R15, R16, R17, R18, R19, R2, R20, R21, R23, R25, R26, R3, R40, R41: symbol GFI_Original:SparkFun_RESISTOR0805-RES -> coreEVSE:SparkFun_RESISTOR0805-RES
- R32, R33, R34, R35, R36, R37, R38, R39: symbol ACTEST_Original:SparkFun-Resistors_0.1OHM-1/2W-1%(1210) -> coreEVSE:SparkFun-Resistors_0.1OHM-1/2W-1%(1210)
- SH1, SH2: footprint OpenEVSE:SHORT_TOP-50 -> coreEVSE:SHORT_TOP-50
- TVS1: footprint OpenEVSE:SMB -> coreEVSE:SMB
- U3: symbol OpenEVSE:MCP9808 -> coreEVSE:MCP9808
- Y1: symbol OpenEVSE:Crystal_16MHz_3.2x2.5mm -> coreEVSE:Crystal_16MHz_3.2x2.5mm

Commit message: end
Parts:
- C28: footprint PCM_SparkFun-Capacitor:C_0805_2012Metric -> PCM_JLCPCB:C_0805
Changed lines of the file:
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@@
 	(wire
 		(pts
+			(xy 67.31 152.4) (xy 74.93 152.4)
+		)
+		(stroke
+			(width 0)
+			(type default)
+		)
+	)
+	(wire
+		(pts
 			(xy 175.26 41.91) (xy 184.15 41.91)
 		)
@@
 	(wire
 		(pts
-			(xy 57.15 137.16) (xy 57.15 140.97)
-		)
-		(stroke
-			(width 0)
-			(type default)
-		)
-	)
-	(wire
-		(pts
 			(xy 85.09 36.83) (xy 90.17 36.83)
 		)
@@
 	(wire
 		(pts
-			(xy 31.75 137.16) (xy 31.75 140.97)
+			(xy 31.75 137.16) (xy 31.75 143.51)
 		)
 		(stroke
@@
 	(wire
 		(pts
-			(xy 60.96 137.16) (xy 57.15 137.16)
-		)
-		(stroke
-			(width 0)
-			(type default)
-		)
-	)
-	(wire
-		(pts
 			(xy 227.33 203.2) (xy 232.41 203.2)
 		)
@@
 		)
 	)
+	(global_label "PE"
+		(shape bidirectional)
+		(at 67.31 152.4 180)
+		(fields_autoplaced yes)
+		(effects
+			(font
+				(size 1.27 1.27)
+			)
+			(justify right)
+		)
+		(property "Intersheetrefs" "${INTERSHEET_REFS}"
+			(at 60.7945 152.4 0)
+			(hide yes)
+			(show_name no)
+			(do_not_autoplace no)
+			(effects
+				(font
+					(size 1.27 1.27)
+				)
+				(justify right)
+			)
+		)
+	)
 	(global_label "ACNIN"
 		(shape bidirectional)
@@
 	(symbol
 		(lib_id "power:GND")
-		(at 31.75 140.97 0)
+		(at 31.75 143.51 0)
 		(unit 1)
 		(body_style 1)
@@
 		(fields_autoplaced yes)
 		(property "Reference" "#PWR039"
-			(at 31.75 147.32 0)
+			(at 31.75 149.86 0)
 			(hide yes)
 			(show_name no)
@@
 		)
 		(property "Value" "GND"
-			(at 31.75 146.05 0)
+			(at 31.75 148.59 0)
 			(show_name no)
 			(do_not_autoplace no)
@@
 		)
 		(property "Footprint" ""
-			(at 31.75 140.97 0)
+			(at 31.75 143.51 0)
 			(hide yes)
 			(show_name no)
@@
 		)
 		(property "Datasheet" ""
-			(at 31.75 140.97 0)
+			(at 31.75 143.51 0)
 			(hide yes)
 			(show_name no)
@@
 		)
 		(property "Description" "Power symbol creates a global label with name \"GND\" , ground"
-			(at 31.75 140.97 0)
+			(at 31.75 143.51 0)
 			(hide yes)
 			(show_name no)
@@
 	(symbol
 		(lib_id "OpenEVSE_PLUS_v6.5.1-eagle-import:HOLE")
-		(at 101.6 139.7 0)
+		(at 115.57 154.94 0)
 		(unit 1)
 		(body_style 1)
@@
 		(dnp no)
 		(property "Reference" "U$3"
-			(at 101.6 139.7 0)
+			(at 115.57 154.94 0)
 			(hide yes)
 			(show_name no)
@@
 		)
 		(property "Value" "HOLE"
-			(at 101.6 139.7 0)
+			(at 115.57 154.94 0)
 			(hide yes)
 			(show_name no)
@@
 		)
 		(property "Footprint" "coreEVSE:HOLE"
-			(at 101.6 139.7 0)
+			(at 115.57 154.94 0)
 			(hide yes)
 			(show_name no)
@@
 		)
 		(property "Datasheet" ""
-			(at 101.6 139.7 0)
+			(at 115.57 154.94 0)
 			(hide yes)
 			(show_name no)
@@
 		)
 		(property "Description" ""
-			(at 101.6 139.7 0)
+			(at 115.57 154.94 0)
 			(hide yes)
 			(show_name no)
@@
 	)
 	(symbol
-		(lib_id "coreEVSE:supply2_PE")
-		(at 57.15 143.51 0)
-		(unit 1)
-		(body_style 1)
-		(exclude_from_sim no)
-		(in_bom yes)
-		(on_board yes)
-		(in_pos_files yes)
-		(dnp no)
-		(property "Reference" "#SUPPLY04"
-			(at 57.15 143.51 0)
-			(hide yes)
-			(show_name no)
-			(do_not_autoplace no)
-			(effects
-				(font
-					(size 1.27 1.27)
-				)
-			)
-		)
-		(property "Value" "PE"
-			(at 55.245 148.209 0)
-			(show_name no)
-			(do_not_autoplace no)
-			(effects
-				(font
-					(size 1.778 1.5113)
-				)
-				(justify left bottom)
-			)
-		)
-		(property "Footprint" ""
-			(at 57.15 143.51 0)
-			(hide yes)
-			(show_name no)
-			(do_not_autoplace no)
-			(effects
-				(font
-					(size 1.27 1.27)
-				)
-			)
-		)
-		(property "Datasheet" ""
-			(at 57.15 143.51 0)
-			(hide yes)
-			(show_name no)
-			(do_not_autoplace no)
-			(effects
-				(font
-					(size 1.27 1.27)
-				)
-			)
-		)
-		(property "Description" "SUPPLY SYMBOL"
-			(at 57.15 143.51 0)
-			(hide yes)
-			(show_name no)
-			(do_not_autoplace no)
-			(effects
-				(font
-					(size 1.27 1.27)
-				)
-			)
-		)
-		(pin "1"
-		)
-		(instances
-			(project "evse"
-				(path "/11cad39f-0746-4064-b162-743100309dbd"
-					(reference "#SUPPLY04")
-					(unit 1)
-				)
-			)
-		)
-	)
-	(symbol
 		(lib_id "power:+5V")
 		(at 370.84 135.89 0)
@@
 			)
 		)
-		(property "Footprint" "PCM_SparkFun-Capacitor:C_0805_2012Metric"
+		(property "Footprint" "PCM_JLCPCB:C_0805"
 			(at 114.3 194.31 0)
 			(hide yes)

Commit message: fix Y1
Parts:
- C1, C2: value 22pF -> 12pF; footprint PCM_JLCPCB:C_0805 -> Capacitor_SMD:C_0402_1005Metric; PROD_ID CAP-25012 -> GRM1555C1H120GA01D; Tolerance 5% -> 2%
- Y1: value 16MHz -> FA-238A 16MHz CL=8pF; footprint PCM_SparkFun-Clock:Crystal_SMD_3.2x2.5mm -> Crystal:Crystal_SMD_SeikoEpson_TSX3225-4Pin_3.2x2.5mm; symbol coreEVSE:Crystal_16MHz_3.2x2.5mm -> coreEVSE:Crystal_GND24; PROD_ID XTAL-14681 -> FA-238A 16.000MHz CL=8pF
Connections:
- net XGND: now also Y1.2 (G), Y1.4 (G)
- net at C1.2, U4.7 (XTAL1/PB6): now also Y1.3; no longer Y1.2
Changed lines of the file:
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@@
 	)
 	(junction
-		(at 205.74 48.26)
-		(diameter 0)
-		(color 0 0 0 0)
-	)
-	(junction
 		(at 129.54 210.82)
 		(diameter 0)
@@
 	)
 	(junction
+		(at 205.74 48.26)
+		(diameter 0)
+		(color 0 0 0 0)
+	)
+	(junction
 		(at 153.67 106.68)
 		(diameter 0)
@@
 	(wire
 		(pts
-			(xy 204.47 48.26) (xy 205.74 48.26)
-		)
-		(stroke
-			(width 0)
-			(type default)
-		)
-	)
-	(wire
-		(pts
 			(xy 175.26 80.01) (xy 184.15 80.01)
 		)
@@
 	(wire
 		(pts
+			(xy 199.39 55.88) (xy 205.74 55.88)
+		)
+		(stroke
+			(width 0)
+			(type default)
+		)
+	)
+	(wire
+		(pts
 			(xy 365.76 198.12) (xy 369.57 198.12)
 		)
@@
 	(wire
 		(pts
-			(xy 203.2 52.07) (xy 203.2 55.88)
-		)
-		(stroke
-			(width 0)
-			(type default)
-		)
-	)
-	(wire
-		(pts
 			(xy 116.84 271.78) (xy 157.48 271.78)
 		)
@@
 	(wire
 		(pts
-			(xy 205.74 48.26) (xy 205.74 49.53)
-		)
-		(stroke
-			(width 0)
-			(type default)
-		)
-	)
-	(wire
-		(pts
 			(xy 82.55 57.15) (xy 85.09 57.15)
 		)
@@
 	(wire
 		(pts
-			(xy 205.74 54.61) (xy 205.74 55.88)
-		)
-		(stroke
-			(width 0)
-			(type default)
-		)
-	)
-	(wire
-		(pts
 			(xy 142.24 208.28) (xy 142.24 210.82)
 		)
@@
 	(wire
 		(pts
+			(xy 199.39 48.26) (xy 205.74 48.26)
+		)
+		(stroke
+			(width 0)
+			(type default)
+		)
+	)
+	(wire
+		(pts
 			(xy 334.01 199.39) (xy 334.01 201.93)
 		)
@@
 	(wire
 		(pts
+			(xy 205.74 48.26) (xy 209.55 48.26)
+		)
+		(stroke
+			(width 0)
+			(type default)
+		)
+	)
+	(wire
+		(pts
 			(xy 264.16 123.19) (xy 265.43 123.19)
 		)
@@
 	(wire
 		(pts
+			(xy 175.26 49.53) (xy 199.39 49.53)
+		)
+		(stroke
+			(width 0)
+			(type default)
+		)
+	)
+	(wire
+		(pts
 			(xy 358.902 27.686) (xy 362.712 27.686)
 		)
@@
 	(wire
 		(pts
+			(xy 199.39 49.53) (xy 199.39 48.26)
+		)
+		(stroke
+			(width 0)
+			(type default)
+		)
+	)
+	(wire
+		(pts
 			(xy 227.33 203.2) (xy 232.41 203.2)
 		)
@@
 	(wire
 		(pts
-			(xy 204.47 49.53) (xy 204.47 48.26)
-		)
-		(stroke
-			(width 0)
-			(type default)
-		)
-	)
-	(wire
-		(pts
 			(xy 153.67 111.76) (xy 153.67 114.3)
 		)
@@
 	(wire
 		(pts
-			(xy 175.26 49.53) (xy 204.47 49.53)
-		)
-		(stroke
-			(width 0)
-			(type default)
-		)
-	)
-	(wire
-		(pts
 			(xy 352.552 31.496) (xy 351.282 31.496)
 		)
@@
 	(wire
 		(pts
-			(xy 321.31 100.33) (xy 327.66 100.33)
+			(xy 199.39 52.07) (xy 199.39 55.88)
 		)
 		(stroke
@@
 	(wire
 		(pts
-			(xy 369.57 210.82) (xy 369.57 209.55)
+			(xy 321.31 100.33) (xy 327.66 100.33)
 		)
 		(stroke
@@
 	(wire
 		(pts
-			(xy 175.26 77.47) (xy 184.15 77.47)
+			(xy 369.57 210.82) (xy 369.57 209.55)
 		)
 		(stroke
@@
 	(wire
 		(pts
-			(xy 22.86 213.36) (xy 22.86 215.9)
+			(xy 175.26 77.47) (xy 184.15 77.47)
 		)
 		(stroke
@@
 	(wire
 		(pts
-			(xy 175.26 52.07) (xy 203.2 52.07)
+			(xy 22.86 213.36) (xy 22.86 215.9)
 		)
 		(stroke
@@
 	(wire
 		(pts
-			(xy 205.74 48.26) (xy 209.55 48.26)
-		)
-		(stroke
-			(width 0)
-			(type default)
-		)
-	)
-	(wire
-		(pts
 			(xy 339.852 70.866) (xy 339.852 78.486)
 		)
@@
 	(wire
 		(pts
-			(xy 203.2 55.88) (xy 205.74 55.88)
-		)
-		(stroke
-			(width 0)
-			(type default)
-		)
-	)
-	(wire
-		(pts
 			(xy 357.632 41.656) (xy 362.712 41.656)
 		)
@@
 	(wire
 		(pts
+			(xy 175.26 52.07) (xy 199.39 52.07)
+		)
+		(stroke
+			(width 0)
+			(type default)
+		)
+	)
+	(wire
+		(pts
 			(xy 379.73 100.33) (xy 386.08 100.33)
 		)
@@
 	(wire
 		(pts
+			(xy 210.82 52.07) (xy 217.17 52.07)
+		)
+		(stroke
+			(width 0)
+			(type default)
+		)
+	)
+	(wire
+		(pts
 			(xy 114.3 195.58) (xy 119.38 195.58)
 		)
@@
 			)
 		)
-		(property "Value" "22pF"
+		(property "Value" "12pF"
 			(at 213.868 60.198 90)
 			(show_name no)
@@
 			)
 		)
-		(property "Footprint" "PCM_JLCPCB:C_0805"
+		(property "Footprint" "Capacitor_SMD:C_0402_1005Metric"
 			(at 200.66 55.88 0)
 			(hide yes)
@@
 			)
 		)
-		(property "Datasheet" "https://cdn.sparkfun.com/assets/8/a/4/a/5/Kemet_Capacitor_Datasheet.pdf"
+		(property "Datasheet" "https://psearch.en.murata.com/capacitor/product/GRM1555C1H120GA01%23.html"
 			(at 195.58 55.88 0)
 			(hide yes)
@@
 			)
 		)
-		(property "Description" "Unpolarized capacitor"
+		(property "Description" "12 pF C0G/NP0 ceramic capacitor, 50 V, 2%, 0402"
 			(at 193.04 55.88 0)
 			(hide yes)
@@
 			)
 		)
-		(property "PROD_ID" "CAP-25012"
+		(property "PROD_ID" "GRM1555C1H120GA01D"
 			(at 198.12 55.88 0)
 			(hide yes)
@@
 			)
 		)
-		(property "Tolerance" "5%"
+		(property "Tolerance" "2%"
 			(at 212.0837 52.07 90)
 			(hide yes)
@@
 	)
 	(symbol
-		(lib_id "coreEVSE:Crystal_16MHz_3.2x2.5mm")
-		(at 205.74 52.07 270)
-		(mirror x)
+		(lib_id "coreEVSE:Crystal_GND24")
+		(at 205.74 52.07 90)
 		(unit 1)
 		(body_style 1)
@@
 			)
 		)
-		(property "Value" "16MHz"
+		(property "Value" "FA-238A 16MHz CL=8pF"
 			(at 214.376 53.594 90)
 			(hide yes)
@@
 			)
 		)
-		(property "Footprint" "PCM_SparkFun-Clock:Crystal_SMD_3.2x2.5mm"
+		(property "Footprint" "Crystal:Crystal_SMD_SeikoEpson_TSX3225-4Pin_3.2x2.5mm"
 			(at 198.12 52.07 0)
 			(hide yes)
@@
 			)
 		)
-		(property "Datasheet" "https://www.murata.com/products/productdata/8801057112094/SPEC-XRCGB16M000FXN01R0.pdf"
+		(property "Datasheet" "https://www.epsondevice.com/crystal/en/products/crystal-unit/fa238a.html"
 			(at 200.66 52.07 0)
 			(hide yes)
@@
 			)
 		)
-		(property "Description" "Crystal"
+		(property "Description" "16 MHz fundamental crystal, CL 8 pF, 4-pad 3225, AEC-Q200"
 			(at 193.04 52.07 0)
 			(hide yes)
@@
 			)
 		)
-		(property "PROD_ID" "XTAL-14681"
+		(property "PROD_ID" "FA-238A 16.000MHz CL=8pF"
 			(at 195.58 52.07 0)
 			(hide yes)
@@
 			)
 		)
-		(property "Value" "22pF"
+		(property "Value" "12pF"
 			(at 215.646 46.99 90)
 			(show_name no)
@@
 			)
 		)
-		(property "Footprint" "PCM_JLCPCB:C_0805"
+		(property "Footprint" "Capacitor_SMD:C_0402_1005Metric"
 			(at 200.66 48.26 0)
 			(hide yes)
@@
 			)
 		)
-		(property "Datasheet" "https://cdn.sparkfun.com/assets/8/a/4/a/5/Kemet_Capacitor_Datasheet.pdf"
+		(property "Datasheet" "https://psearch.en.murata.com/capacitor/product/GRM1555C1H120GA01%23.html"
 			(at 195.58 48.26 0)
 			(hide yes)
@@
 			)
 		)
-		(property "Description" "Unpolarized capacitor"
+		(property "Description" "12 pF C0G/NP0 ceramic capacitor, 50 V, 2%, 0402"
 			(at 193.04 48.26 0)
 			(hide yes)
@@
 			)
 		)
-		(property "PROD_ID" "CAP-25012"
+		(property "PROD_ID" "GRM1555C1H120GA01D"
 			(at 198.12 48.26 0)
 			(hide yes)
@@
 			)
 		)
-		(property "Tolerance" "5%"
+		(property "Tolerance" "2%"
 			(at 212.0837 44.45 90)
 			(hide yes)

Commit message: fix SH3
Parts:
- added SH3: NetTie_2, NetTie:NetTie-2_SMD_Pad0.5mm, symbol Device:NetTie_2
- SH1, SH2: footprint coreEVSE:SHORT_TOP-50 -> NetTie:NetTie-2_SMD_Pad0.5mm
Connections:
- net GND: now also SH3.1
- net PE: now also SH3.2
Changed lines of the file:
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@@
 	(wire
 		(pts
+			(xy 267.97 72.39) (xy 270.51 72.39)
+		)
+		(stroke
+			(width 0)
+			(type default)
+		)
+	)
+	(wire
+		(pts
 			(xy 259.08 63.5) (xy 267.97 63.5)
 		)
@@
 		)
 	)
+	(global_label "PE"
+		(shape bidirectional)
+		(at 275.59 72.39 0)
+		(fields_autoplaced yes)
+		(effects
+			(font
+				(size 1.27 1.27)
+			)
+			(justify left)
+		)
+		(property "Intersheetrefs" "${INTERSHEET_REFS}"
+			(at 282.1055 72.39 0)
+			(hide yes)
+			(show_name no)
+			(do_not_autoplace no)
+			(effects
+				(font
+					(size 1.27 1.27)
+				)
+				(justify left)
+			)
+		)
+	)
 	(global_label "DC_RELAY_1"
 		(shape bidirectional)
@@
 			)
 		)
-		(property "Footprint" "coreEVSE:SHORT_TOP-50"
+		(property "Footprint" "NetTie:NetTie-2_SMD_Pad0.5mm"
 			(at 222.25 52.07 0)
 			(hide yes)
@@
 			)
 		)
-		(property "Footprint" "coreEVSE:SHORT_TOP-50"
+		(property "Footprint" "NetTie:NetTie-2_SMD_Pad0.5mm"
 			(at 153.67 109.22 0)
 			(hide yes)
@@
 					(unit 1)
 				)
+			)
+		)
+	)
+	(symbol
+		(lib_id "Device:NetTie_2")
+		(at 273.05 72.39 0)
+		(unit 1)
+		(body_style 1)
+		(exclude_from_sim no)
+		(in_bom no)
+		(on_board yes)
+		(in_pos_files yes)
+		(dnp no)
+		(property "Reference" "SH3"
+			(at 273.05 69.85 0)
+			(show_name no)
+			(do_not_autoplace no)
+			(effects
+				(font
+					(size 1.27 1.27)
+				)
+			)
+		)
+		(property "Value" "NetTie_2"
+			(at 273.05 74.93 0)
+			(hide yes)
+			(show_name no)
+			(do_not_autoplace no)
+			(effects
+				(font
+					(size 1.27 1.27)
+				)
+			)
+		)
+		(property "Footprint" "NetTie:NetTie-2_SMD_Pad0.5mm"
+			(at 273.05 72.39 0)
+			(hide yes)
+			(show_name no)
+			(do_not_autoplace no)
+			(effects
+				(font
+					(size 1.27 1.27)
+				)
+			)
+		)
+		(property "Datasheet" ""
+			(at 273.05 72.39 0)
+			(hide yes)
+			(show_name no)
+			(do_not_autoplace no)
+			(effects
+				(font
+					(size 1.27 1.27)
+				)
+			)
+		)
+		(property "Description" "Single-point PE to electronics GND reference bond for Control Pilot"
+			(at 273.05 72.39 0)
+			(hide yes)
+			(show_name no)
+			(do_not_autoplace no)
+			(effects
+				(font
+					(size 1.27 1.27)
+				)
+			)
+		)
+		(pin "1"
+		)
+		(pin "2"
+		)
+		(instances
+			(project "evse"
+				(path "/11cad39f-0746-4064-b162-743100309dbd"
+					(reference "SH3")
+					(unit 1)
+				)

Commit message: done
Parts:
- removed U$3, U$9: HOLE, coreEVSE:HOLE, symbol OpenEVSE_PLUS_v6.5.1-eagle-import:HOLE
- added R42, R43: 47k, Resistor_SMD:R_0805_2012Metric, symbol coreEVSE:SparkFun_RESISTOR0805-RES
- C10, C13, C26, C5, C6: footprint Capacitor_SMD:C_0805_2012Metric -> Capacitor_SMD:C_1210_3225Metric; PROD_ID TBD-10uF-10V-X7R-0603 -> C3225X7R1H106K250AC; Tolerance 20% -> 10%; Voltage 10V -> 50V
- D10, D7, D8, D9: value 1N4004 -> S1M; PROD_ID (none) -> S1M-13-F
- R32, R33, R34, R35, R36, R37, R38, R39: footprint Resistor_SMD:R_1210_3225Metric -> Resistor_SMD:R_2512_6332Metric; Creepage (none) -> >=4.5 mm along top of 2512 body between terminations; PCB c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; MPN (none) -> HV733ATTE1803F; Manufacturer (none) -> KOA Speer; Max working voltage (none) -> 3000 VDC absolute; 424 VDC rated at 180k; Overload (none) -> 1061 VDC for 5 s at 180k; 4000 VDC absolute maximum; PROD_ID RES-12374 -> (none); Power (none) -> 1 W @ 70C; Pulse (none) -> One-pulse limiting-power curve in KOA HV73 datasheet; max a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; Tolerance (none) -> 1%
Connections:
- net GND: now also U3.5 (A2), U3.6 (A1), U3.7 (A0), R42.2, R43.1
- net at Q2.1 (B), R24.1: now also R42.1
- net at Q3.1 (B), R11.2: now also R43.2
- no-connect marks 11 -> 8
Other:
- moved on the sheet: Pilot1

Commit message: tested
Parts:
- C21: footprint PCM_SparkFun-Capacitor:C_0805_2012Metric -> PCM_JLCPCB:C_0805
- U2: value TC1044S -> LTC1144IS8#TRPBF; symbol Regulator_SwitchedCapacitor:LTC1044 -> coreEVSE:LTC1144
Connections:
- net ACLIN: now also F1.1; no longer PS1.2 (AC/L)
- net ACNIN: now also PS1.1 (AC/N); no longer F1.1
- net at F1.2: now also PS1.2 (AC/L); no longer PS1.1 (AC/N)
Other:
- note added: "230 V AC RMS between ACLIN (L) and ACNIN (N)"
- moved on the sheet: F1
