File: evse.kicad_sch (KiCad schematic)
At the start: 118 parts, among them IC1 LF353, IC3 LM358, IC8 HCPL-2731S, J1 ISP, J4 T44009, J5 T44009, J6 T44009, J7 T44009, J8 T44009, J9 T44009, K1 HF186F/12-HCTF, K2 HF186F/12-HCTF, M1 MOV, M2 MOV, M3 MOV, Q2 MMBT2222A, Q3 MMBT2222A, U1 AP63205WU, U2 LTC1144IS8#TRPBF, U3 MCP9808, U4 ATmega328P-AU, Y1 FA-238A 16MHz CL=8pF

Commit message: new
Parts:
- removed C22: 10uF, Capacitor_SMD:C_1206_3216Metric, symbol PCM_SparkFun-Capacitor:1.0uF_0805_25V_10%
- removed C23, C24: 1.0uF, PCM_SparkFun-Capacitor:C_0805_2012Metric, symbol PCM_SparkFun-Capacitor:1.0uF_0805_25V_10%
- removed C28: 10uF, PCM_JLCPCB:C_0805, symbol PCM_SparkFun-Capacitor:1.0uF_0805_25V_10%
- removed C29, C33: 22uF, PCM_SparkFun-Capacitor:C_0805_2012Metric, symbol PCM_SparkFun-Capacitor:22uF_0805_16V_20%
- removed C32: 0.1uF, Capacitor_SMD:C_0805_2012Metric, symbol PCM_SparkFun-Capacitor:0.1uF_0402_16V_10%
- removed D2, D5: SS14, Diode_SMD:D_SOD-123, symbol Diode:1N4148W
- removed F1: 1.6A 250VAC slow-blow, coreEVSE:BELFUSE1A, symbol PCM_SparkFun-Fuse:Fuse
- removed L2: 4.7uH, coreEVSE:NR5040, symbol PCM_SparkFun-Coil:3.3uH_0805_0.45A
- removed PS1: IRM-10-12, coreEVSE:Converter_ACDC_MeanWell_IRM-10-12_THT, symbol Converter_ACDC:IRM-10-12
- removed Q2, Q3: MMBT2222A, Package_TO_SOT_SMD:SOT-23, symbol Transistor_BJT:MMBT2222A
- removed R11, R24: 220, Resistor_SMD:R_0805_2012Metric, symbol PCM_SparkFun-Resistor:330_0402
- removed R42, R43: 47k, Resistor_SMD:R_0805_2012Metric, symbol coreEVSE:SparkFun_RESISTOR0805-RES
- removed U1: AP63205WU, Package_TO_SOT_SMD:TSOT-23-6, symbol Regulator_Switching:AP63205WU
Other:
- added sheet Power Supplies (power_supplies.kicad_sch)
- added sheet Relay Control (relay_control.kicad_sch)
- note removed: "Power +12V"
- note removed: "Power +12V to +5V"
- note removed: "Relay Control"

Commit message: fix
Parts:
- removed C10, C13, C26, C5, C6: 10uF, Capacitor_SMD:C_1210_3225Metric, symbol PCM_SparkFun-Capacitor:1.0uF_0805_25V_10%
- removed C11: 0.1uF, Capacitor_SMD:C_0805_2012Metric, symbol coreEVSE:SparkFun_CAP0805
- removed C14: 10uf, coreEVSE:C_1206_3216Metric_AC, symbol coreEVSE:SparkFun_CAP_POL1206
- removed C15: 1.0uF, PCM_SparkFun-Capacitor:C_0805_2012Metric, symbol PCM_SparkFun-Capacitor:1.0uF_0805_25V_10%
- removed C16, C7: .1uf, Capacitor_SMD:C_0805_2012Metric, symbol coreEVSE:SparkFun_CAP0805
- removed C34: 100nF, Capacitor_SMD:C_0805_2012Metric, symbol coreEVSE:SparkFun_CAP0805
- removed CurrentCoil1: KF128-2.54-2P, coreEVSE:TerminalBlock_KF128-2.54-2P, symbol coreEVSE:KF128-2.54-2P
- removed D1: AZ23C5V6-7-F, Package_TO_SOT_SMD:SOT-23, symbol coreEVSE:diode_BAS40-06
- removed D10, D7, D8, D9: S1M, coreEVSE:SMA_AC, symbol coreEVSE:diode_MBRA340T3
- removed D11: AZ23C2V7, PCM_SparkFun-Semiconductor-Standard:SOT23-3, symbol coreEVSE:diode_BAS40-06
- removed D3, D4, D6: 1N4148, coreEVSE:SOD-123_AC, symbol coreEVSE:diode_DIODE-SOD123
- removed GFCI_CT1: KF128-2.54-4P, coreEVSE:TerminalBlock_KF128-2.54-4P, symbol coreEVSE:KF128-2.54-4P
- removed IC1: LF353, Package_SO:SOIC-8_3.9x4.9mm_P1.27mm, symbol Amplifier_Operational:LMV358
- removed IC3: LM358, Package_SO:SOIC-8_3.9x4.9mm_P1.27mm, symbol coreEVSE:SparkFun_LMV358
- removed IC8: HCPL-2731S, coreEVSE:SIL8-2, symbol coreEVSE:OpenEVSE_HCPL-2731S
- removed K1, K2: HF186F/12-HCTF, coreEVSE:Relay_Hongfa_HF186F_PushIn, symbol coreEVSE:HF186F
- removed R1: 620, Resistor_SMD:R_0805_2012Metric, symbol PCM_SparkFun-Resistor:10k_0402
- removed R14, R16, R21, R25: 100k, Resistor_SMD:R_0805_2012Metric, symbol coreEVSE:SparkFun_RESISTOR0805-RES
- removed R15: 20k, Resistor_SMD:R_0805_2012Metric, symbol coreEVSE:SparkFun_RESISTOR0805-RES
- removed R17: 422, Resistor_SMD:R_0805_2012Metric, symbol coreEVSE:SparkFun_RESISTOR0805-RES
- removed R18: 100, Resistor_SMD:R_0805_2012Metric, symbol coreEVSE:SparkFun_RESISTOR0805-RES
- removed R19, R2: 10k, Resistor_SMD:R_0805_2012Metric, symbol coreEVSE:SparkFun_RESISTOR0805-RES
- removed R20, R3: 1k, Resistor_SMD:R_0805_2012Metric, symbol coreEVSE:SparkFun_RESISTOR0805-RES
- removed R23: 330, Resistor_SMD:R_0805_2012Metric, symbol coreEVSE:SparkFun_RESISTOR0805-RES
- removed R26: 20R 1% 0.25W, Resistor_SMD:R_0805_2012Metric, symbol coreEVSE:SparkFun_RESISTOR0805-RES
- removed R32, R33, R34, R35, R36, R37, R38, R39: 180k, Resistor_SMD:R_2512_6332Metric, symbol coreEVSE:SparkFun-Resistors_0.1OHM-1/2W-1%(1210)
- removed R40, R41: 4.7k, Resistor_SMD:R_0805_2012Metric, symbol coreEVSE:SparkFun_RESISTOR0805-RES
- removed R5: 56k, Resistor_SMD:R_0805_2012Metric, symbol PCM_SparkFun-Resistor:10k_0402
- removed R6, R8, R9: 100k, Resistor_SMD:R_0805_2012Metric, symbol PCM_SparkFun-Resistor:10k_0402
- removed R7: 200k, Resistor_SMD:R_0805_2012Metric, symbol PCM_SparkFun-Resistor:10k_0402
- removed TVS1: P6SMB16CA, coreEVSE:SMB, symbol Device:D_TVS
- removed U2: LTC1144IS8#TRPBF, Package_SO:SOIC-8_3.9x4.9mm_P1.27mm, symbol coreEVSE:LTC1144
- removed U3: MCP9808, Package_SO:MSOP-8_3x3mm_P0.65mm, symbol coreEVSE:MCP9808
- C1, C2: symbol PCM_SparkFun-Capacitor:22pF_0402_50V_5% -> coreEVSE:JLCPCB_C_small; LCSC (none) -> C696888
- C12, C19, C27: footprint PCM_SparkFun-Capacitor:C_0805_2012Metric -> Capacitor_SMD:C_0805_2012Metric; symbol PCM_SparkFun-Capacitor:0.1uF_0402_16V_10% -> coreEVSE:JLCPCB_C_100n; LCSC (none) -> C129641
- C20, C3, C4, C9: footprint PCM_SparkFun-Capacitor:C_0805_2012Metric -> Capacitor_SMD:C_0805_2012Metric; symbol PCM_SparkFun-Capacitor:1.0uF_0805_25V_10% -> coreEVSE:JLCPCB_C_1u; LCSC (none) -> C3848979
- C21: footprint PCM_JLCPCB:C_0805 -> Capacitor_SMD:C_0805_2012Metric; symbol PCM_SparkFun-Capacitor:0.1uF_0402_16V_10% -> coreEVSE:JLCPCB_C_100n; LCSC (none) -> C129641
- C35: symbol PCM_SparkFun-Capacitor:0.1uF_0402_16V_10% -> coreEVSE:JLCPCB_C_100n; LCSC (none) -> C169842
- FID1, FID2, FID3, FID4: symbol OpenEVSE_PLUS_v6.5.1-eagle-import:FIDUCIAL1X2.5 -> Mechanical:Fiducial; now left out of the parts list
- L1: footprint PCM_SparkFun-Coil:0805 -> Inductor_SMD:L_0805_2012Metric; LCSC (none) -> C74764
- R10, R22, R31: symbol PCM_SparkFun-Resistor:10k_0402 -> coreEVSE:JLCPCB_R_a; LCSC (none) -> C7337170
- R27: symbol PCM_SparkFun-Resistor:10k_0402 -> coreEVSE:JLCPCB_R_a; LCSC (none) -> C2078467
Connections:
- net UGND: now also C12.2, C20.1; no longer C12.1, C20.2
- net AC_L_OUT renamed ACLOUT
- net AC_N_OUT renamed ACNOUT
- removed net AREF: C12.2, C20.1, U4.20 (AREF)
- new net: C12.1, C20.2, U4.20 (AREF)
- no-connect marks 8 -> 3
Other:
- added sheet Current and GFI Monitoring (gfi.kicad_sch)
- added sheet PP Read (pp.kicad_sch)
- added sheet Pilot (pilot.kicad_sch)
- added sheet Temperature Monitoring (temperature_monitoring.kicad_sch)
- added sheet Weld Detect (weld.kicad_sch)
- note removed: "230 V AC RMS between ACLIN (L) and ACNIN (N)"
- note removed: "AMP CT: OPCT16AL-1000/1, 100 A / 100 mA Pass ONE power conductor through core"
- note removed: "CURRENT READ"
- note removed: "Fault"
- note removed: "GFCI CT: OpenEVSE / CR8420-1000-G custom 4 wires: sense winding + 5-turn self-test winding"
- note removed: "GFI"
- note removed: "PILOT"
- note removed: "PP Read"
- note removed: "Temperature sensor"
- note removed: "WELD DETECT"
- moved on the sheet: C1, C12, C17, C18, C19, C2, C20, C21, C27, C3, C35, C4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
