File: power_supplies.kicad_sch (KiCad schematic)
At the start: 11 parts, among them U1 AP63205WU

Commit message: fix
Parts:
- C22: symbol PCM_SparkFun-Capacitor:1.0uF_0805_25V_10% -> coreEVSE:JLCPCB_C_1u; LCSC (none) -> C380364
- C23, C24: footprint PCM_SparkFun-Capacitor:C_0805_2012Metric -> Capacitor_SMD:C_0805_2012Metric; symbol PCM_SparkFun-Capacitor:1.0uF_0805_25V_10% -> coreEVSE:JLCPCB_C_1u; LCSC (none) -> C3848979
- C28: footprint PCM_JLCPCB:C_0805 -> Capacitor_SMD:C_0805_2012Metric; symbol PCM_SparkFun-Capacitor:1.0uF_0805_25V_10% -> coreEVSE:JLCPCB_C_1u; LCSC (none) -> C5448891
- C29, C33: footprint PCM_SparkFun-Capacitor:C_0805_2012Metric -> Capacitor_SMD:C_0805_2012Metric; symbol PCM_SparkFun-Capacitor:22uF_0805_16V_20% -> coreEVSE:JLCPCB_C_22u; LCSC (none) -> C380339
- C32: symbol PCM_SparkFun-Capacitor:0.1uF_0402_16V_10% -> coreEVSE:JLCPCB_C_100n; LCSC (none) -> C129641
- L2: symbol PCM_SparkFun-Coil:3.3uH_0805_0.45A -> coreEVSE:JLCPCB_L_generic; LCSC (none) -> C2045677
