File: relay_control.kicad_sch (KiCad schematic)
At the start: 8 parts, among them Q2 MMBT2222A, Q3 MMBT2222A

Commit message: fix
Parts:
- added K1, K2: HF186F/12-HTF, coreEVSE:Relay_Hongfa_HF186F_PushIn, symbol coreEVSE:HF186F
- D2, D5: value SS14 -> B5819W; symbol Diode:1N4148W -> coreEVSE:D_Schottky; LCSC (none) -> C64885
- Q2, Q3: value MMBT2222A -> AO3400A; symbol Transistor_BJT:MMBT2222A -> coreEVSE:AO3400A; LCSC (none) -> C2803353
- R11, R24: symbol PCM_SparkFun-Resistor:330_0402 -> coreEVSE:JLCPCB_R_b; LCSC (none) -> C17557
- R42, R43: symbol coreEVSE:SparkFun_RESISTOR0805-RES -> coreEVSE:JLCPCB_R_generic; LCSC (none) -> C4238470
Connections:
- net +12V: now also K1.A2, K2.A2
- net DC_RELAY_C1: now also K1.A1
- net DC_RELAY_C2: now also K2.A1
- new net ACLIN: K1.14
- new net ACLOUT: K1.13
- new net ACNIN: K2.14
- new net ACNOUT: K2.13
