File: _restore_backup_2026-09-21T01-21-14-846/evse.kicad_pcb (KiCad board)
At the start: 2 copper layers, 100 x 100 mm, 117 parts, among them IC1 LF353, IC2 ATmega328P, IC3 LM358, IC8 HCPL-2731S, J1 ISP, J4 T44009, J5 T44009, J6 T44009, J7 T44009, J8 T44009, J9 T44009, K1 HF186F/12-HCTF, K2 HF186F/12-HCTF, M1 MOV-20D431K, M2 MOV-20D431K, M3 MOV-20D431K, Q2 MMBT2222A, Q3 MMBT2222A, U1 AP63205WU, U2 TC1044S, U3 MCP9808, Y1 16MHz

Commit message: 21/09
Parts:
- moved J5 1.00 mm to (28.0, 92.0)
Other:
- outline, holes or cut-outs redrawn
