File: _restore_backup_2026-09-21T01-21-14-846/evse.kicad_sch (KiCad schematic)
At the start: 111 parts, among them IC1 LF353, IC2 ATmega328P, IC3 LM358, IC8 HCPL-2731S, J1 ISP, J4 T44009, J5 T44009, J6 T44009, J7 T44009, J8 T44009, J9 T44009, K1 HF186F/12-HCTF, K2 HF186F/12-HCTF, M1 MOV, M2 MOV, M3 MOV, Q2 MMBT2222A, Q3 MMBT2222A, U1 AP63205WU, U2 TC1044S, U3 MCP9808, Y1 16MHz

Commit message: 21/09
Parts:
- M1, M2, M3: value MOV -> MOV-20D431K; footprint OpenEVSE:MOV -> Bourns:MOV-20D431K_Horizontal; symbol MOV_Original:OpenEVSE_MOV -> Bourns:MOV-20D431K; MPN (none) -> MOV-20D431K; Manufacturer (none) -> Bourns
Connections:
- net ACLIN: now also M1.1, M3.1; no longer M1.P$1 (1), M3.P$1 (1)
- net ACNIN: now also M1.2, M2.1; no longer M1.P$2 (2), M2.P$1 (1)
- net PE: now also M2.2, M3.2; no longer M2.P$2 (2), M3.P$2 (2)
Changed lines of the file:
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@@
 	)
 	(symbol
-		(lib_id "MOV_Original:OpenEVSE_MOV")
+		(lib_id "Bourns:MOV-20D431K")
 		(at 353.06 204.47 90)
 		(unit 1)
@@
 			)
 		)
-		(property "Value" "MOV"
+		(property "Value" "MOV-20D431K"
 			(at 350.774 207.264 0)
 			(show_name no)
@@
 			)
 		)
-		(property "Footprint" "OpenEVSE:MOV"
+		(property "Footprint" "Bourns:MOV-20D431K_Horizontal"
 			(at 353.06 204.47 0)
 			(hide yes)
@@
 			)
 		)
-		(property "Datasheet" ""
+		(property "Datasheet" "https://www.bourns.com/docs/product-datasheets/mov20d.pdf"
 			(at 353.06 204.47 0)
 			(hide yes)
@@
 			)
 		)
-		(property "Description" ""
+		(property "Description" "Bourns 20 mm MOV; 275 VAC, 350 VDC, Vvar 430 V +/-10%, clamp 710 V, 6.5 kA, 190 J"
+			(at 353.06 204.47 0)
+			(hide yes)
+			(show_name no)
+			(do_not_autoplace no)
+			(effects
+				(font
+					(size 1.27 1.27)
+				)
+			)
+		)
+		(property "Manufacturer" "Bourns"
 			(at 353.06 204.47 0)
+			(show_name no)
+			(do_not_autoplace no)
 			(hide yes)
+			(effects
+				(font
+					(size 1.27 1.27)
+				)
+			)
+		)
+		(property "MPN" "MOV-20D431K"
+			(at 353.06 204.47 0)
 			(show_name no)
 			(do_not_autoplace no)
+			(hide yes)
 			(effects
 				(font
@@
 			)
 		)
-		(pin "P$2"
+		(pin "2"
 		)
-		(pin "P$1"
+		(pin "1"
 		)
 		(instances
@@
 	)
 	(symbol
-		(lib_id "MOV_Original:OpenEVSE_MOV")
+		(lib_id "Bourns:MOV-20D431K")
 		(at 386.08 204.47 90)
 		(unit 1)
@@
 			)
 		)
-		(property "Value" "MOV"
+		(property "Value" "MOV-20D431K"
 			(at 383.794 207.264 0)
 			(show_name no)
@@
 			)
 		)
-		(property "Footprint" "OpenEVSE:MOV"
+		(property "Footprint" "Bourns:MOV-20D431K_Horizontal"
 			(at 386.08 204.47 0)
 			(hide yes)
@@
 			)
 		)
-		(property "Datasheet" ""
+		(property "Datasheet" "https://www.bourns.com/docs/product-datasheets/mov20d.pdf"
 			(at 386.08 204.47 0)
 			(hide yes)
@@
 			)
 		)
-		(property "Description" ""
+		(property "Description" "Bourns 20 mm MOV; 275 VAC, 350 VDC, Vvar 430 V +/-10%, clamp 710 V, 6.5 kA, 190 J"
+			(at 386.08 204.47 0)
+			(hide yes)
+			(show_name no)
+			(do_not_autoplace no)
+			(effects
+				(font
+					(size 1.27 1.27)
+				)
+			)
+		)
+		(property "Manufacturer" "Bourns"
 			(at 386.08 204.47 0)
+			(show_name no)
+			(do_not_autoplace no)
 			(hide yes)
+			(effects
+				(font
+					(size 1.27 1.27)
+				)
+			)
+		)
+		(property "MPN" "MOV-20D431K"
+			(at 386.08 204.47 0)
 			(show_name no)
 			(do_not_autoplace no)
+			(hide yes)
 			(effects
 				(font
@@
 			)
 		)
-		(pin "P$2"
+		(pin "2"
 		)
-		(pin "P$1"
+		(pin "1"
 		)
 		(instances
@@
 	)
 	(symbol
-		(lib_id "MOV_Original:OpenEVSE_MOV")
+		(lib_id "Bourns:MOV-20D431K")
 		(at 369.57 204.47 90)
 		(unit 1)
@@
 			)
 		)
-		(property "Value" "MOV"
+		(property "Value" "MOV-20D431K"
 			(at 367.284 207.264 0)
 			(show_name no)
@@
 			)
 		)
-		(property "Footprint" "OpenEVSE:MOV"
+		(property "Footprint" "Bourns:MOV-20D431K_Horizontal"
 			(at 369.57 204.47 0)
 			(hide yes)
@@
 			)
 		)
-		(property "Datasheet" ""
+		(property "Datasheet" "https://www.bourns.com/docs/product-datasheets/mov20d.pdf"
 			(at 369.57 204.47 0)
 			(hide yes)
@@
 			)
 		)
-		(property "Description" ""
+		(property "Description" "Bourns 20 mm MOV; 275 VAC, 350 VDC, Vvar 430 V +/-10%, clamp 710 V, 6.5 kA, 190 J"
+			(at 369.57 204.47 0)
+			(hide yes)
+			(show_name no)
+			(do_not_autoplace no)
+			(effects
+				(font
+					(size 1.27 1.27)
+				)
+			)
+		)
+		(property "Manufacturer" "Bourns"
 			(at 369.57 204.47 0)
+			(show_name no)
+			(do_not_autoplace no)
 			(hide yes)
+			(effects
+				(font
+					(size 1.27 1.27)
+				)
+			)
+		)
+		(property "MPN" "MOV-20D431K"
+			(at 369.57 204.47 0)
 			(show_name no)
 			(do_not_autoplace no)
+			(hide yes)
 			(effects
 				(font
@@
 			)
 		)
-		(pin "P$2"
+		(pin "2"
 		)
-		(pin "P$1"
+		(pin "1"
 		)
 		(instances
